File: hdw/LTC7851_Demo/POS5_Control.sch (KiCad schematic (older format))
At the start: 7 parts

Commit message: Added component values for all phase 1 components
Parts:
- removed C?: C, symbol Custom_Library:C_Custom
- removed R? (x3): R, symbol Custom_Library:R_Custom
- added C? (x2): 0.1uF, symbol Custom_Library:C_Custom
- added R? (x2): 2, symbol Custom_Library:R_Custom
- R?: value R -> 51.1k; Tolerance Tol -> 1%; Wattage W -> 1/10W; display_footprint Foot -> 0603
Connections:
- wire segments 17 -> 16
Changed lines of the file:
@@
 $Descr A 11000 8500
 encoding utf-8
-Sheet 3 15
+Sheet 3 14
 Title ""
 Date ""
@@
 AR Path="/5BB86F26/5BBB20F1" Ref="R?"  Part="1"
 F 0 "R?" H 2820 5780 50  0000 R CNN
-F 1 "R" V 2920 5780 50  0000 C CNN
+F 1 "51.1k" V 2920 5780 40  0000 C CNN
 F 2 "" H 2920 5780 50  0001 C CNN
 F 3 "" H 2920 5780 50  0001 C CNN
 F 4 "PN" H 3220 6180 60  0001 C CNN "Digi-Key PN"
-F 5 "Foot" H 3020 5860 50  0000 L CNN "display_footprint"
-F 6 "Tol" H 3020 5780 50  0000 L CNN "Tolerance"
-F 7 "W" H 3020 5700 50  0000 L CNN "Wattage"
+F 5 "0603" H 3020 5860 50  0000 L CNN "display_footprint"
+F 6 "1%" H 3020 5780 50  0000 L CNN "Tolerance"
+F 7 "1/10W" H 3020 5700 50  0000 L CNN "Wattage"
 	1    2920 5780
 	-1   0    0    -1
@@
 	2920 5560 3000 5560
 $Comp
-L Custom_Library:R_Custom R?
-U 1 1 5BBB2173
-P 2780 2730
-AR Path="/5BB86F29/5BBB2173" Ref="R?"  Part="1"
-AR Path="/5BB9CE4B/5BBB2173" Ref="R?"  Part="1"
-AR Path="/5BB86F26/5BBB2173" Ref="R?"  Part="1"
-F 0 "R?" H 2680 2730 50  0000 R CNN
-F 1 "R" V 2780 2730 50  0000 C CNN
-F 2 "" H 2780 2730 50  0001 C CNN
-F 3 "" H 2780 2730 50  0001 C CNN
-F 4 "PN" H 3080 3130 60  0001 C CNN "Digi-Key PN"
-F 5 "Foot" H 2880 2810 50  0000 L CNN "display_footprint"
-F 6 "Tol" H 2880 2730 50  0000 L CNN "Tolerance"
-F 7 "W" H 2880 2650 50  0000 L CNN "Wattage"
-	1    2780 2730
-	1    0    0    -1
-$EndComp
-$Comp
-L Custom_Library:R_Custom R?
-U 1 1 5BBB222D
-P 2780 3280
-AR Path="/5BB86F29/5BBB222D" Ref="R?"  Part="1"
-AR Path="/5BB9CE4B/5BBB222D" Ref="R?"  Part="1"
-AR Path="/5BB86F26/5BBB222D" Ref="R?"  Part="1"
-F 0 "R?" H 2680 3280 50  0000 R CNN
-F 1 "R" V 2780 3280 50  0000 C CNN
-F 2 "" H 2780 3280 50  0001 C CNN
-F 3 "" H 2780 3280 50  0001 C CNN
-F 4 "PN" H 3080 3680 60  0001 C CNN "Digi-Key PN"
-F 5 "Foot" H 2880 3360 50  0000 L CNN "display_footprint"
-F 6 "Tol" H 2880 3280 50  0000 L CNN "Tolerance"
-F 7 "W" H 2880 3200 50  0000 L CNN "Wattage"
-	1    2780 3280
-	1    0    0    -1
-$EndComp
-Wire Wire Line
-	2780 3130 2780 3010
-Wire Wire Line
-	2780 3010 3000 3010
-Wire Wire Line
-	2780 3010 2780 2880
-Connection ~ 2780 3010
-$Comp
-L power:GND #PWR?
-U 1 1 5BBB2378
-P 2780 3430
-F 0 "#PWR?" H 2780 3180 50  0001 C CNN
-F 1 "GND" H 2780 3280 50  0000 C CNN
-F 2 "" H 2780 3430 50  0001 C CNN
-F 3 "" H 2780 3430 50  0001 C CNN
-	1    2780 3430
-	1    0    0    -1
-$EndComp
-$Comp
 L power:+12V #PWR?
 U 1 1 5BBB23BE
-P 2780 2580
-F 0 "#PWR?" H 2780 2430 50  0001 C CNN
-F 1 "+12V" H 2780 2720 50  0000 C CNN
-F 2 "" H 2780 2580 50  0001 C CNN
-F 3 "" H 2780 2580 50  0001 C CNN
-	1    2780 2580
-	1    0    0    -1
-$EndComp
-$Comp
-L Custom_Library:C_Custom C?
-U 1 1 5BBB265D
-P 2780 1990
-F 0 "C?" H 2805 2090 50  0000 L CNN
-F 1 "C" H 2805 1890 50  0000 L CNN
-F 2 "" H 2818 1840 50  0001 C CNN
-F 3 "" H 2805 2090 50  0001 C CNN
-F 4 "Foot" H 2630 2090 50  0000 R CNN "display_footprint"
-F 5 "V" H 2630 1990 50  0000 R CNN "Voltage"
-F 6 "Er" H 2630 1890 50  0000 R CNN "Dielectric"
-F 7 "PN" H 3205 2490 60  0001 C CNN "Digi-Key PN"
-	1    2780 1990
-	1    0    0    -1
-$EndComp
-$Comp
-L power:GND #PWR?
-U 1 1 5BBB26FB
-P 2780 2140
-F 0 "#PWR?" H 2780 1890 50  0001 C CNN
-F 1 "GND" H 2780 1990 50  0000 C CNN
-F 2 "" H 2780 2140 50  0001 C CNN
-F 3 "" H 2780 2140 50  0001 C CNN
-	1    2780 2140
-	1    0    0    -1
-$EndComp
-Wire Wire Line
-	2780 1840 2780 1760
-Wire Wire Line
-	2780 1760 3000 1760
-$Comp
-L Custom_Library:R_Custom R?
-U 1 1 5BBB2A4A
-P 2320 1760
-F 0 "R?" V 2220 1760 50  0000 C CNN
-F 1 "R" V 2320 1760 50  0000 C CNN
-F 2 "" H 2320 1760 50  0001 C CNN
-F 3 "" H 2320 1760 50  0001 C CNN
-F 4 "Foot" V 2420 1760 50  0000 C CNN "display_footprint"
-F 5 "Tol" V 2520 1760 50  0000 C CNN "Tolerance"
-F 6 "W" V 2620 1760 50  0000 C CNN "Wattage"
-F 7 "PN" H 2620 2160 60  0001 C CNN "Digi-Key PN"
-	1    2320 1760
-	0    1    1    0
-$EndComp
-Wire Wire Line
-	2470 1760 2780 1760
-Connection ~ 2780 1760
+P 2780 2590
+F 0 "#PWR?" H 2780 2440 50  0001 C CNN
+F 1 "+12V" H 2780 2730 50  0000 C CNN
+F 2 "" H 2780 2590 50  0001 C CNN
+F 3 "" H 2780 2590 50  0001 C CNN
+	1    2780 2590
+	1    0    0    -1
+$EndComp
 $Comp
 L Custom_Library:+5.5V_MNG #PWR?
 U 1 1 5BBB2BF1
-P 1960 1680
-F 0 "#PWR?" H 1960 1530 50  0001 C CNN
-F 1 "+5.5V_MNG" H 1960 1820 50  0000 C CNN
-F 2 "" H 1960 1680 50  0001 C CNN
-F 3 "" H 1960 1680 50  0001 C CNN
-	1    1960 1680
-	1    0    0    -1
-$EndComp
-Wire Wire Line
-	1960 1680 1960 1760
-Wire Wire Line
-	1960 1760 2170 1760
+P 2780 1260
+F 0 "#PWR?" H 2780 1110 50  0001 C CNN
+F 1 "+5.5V_MNG" H 2780 1400 50  0000 C CNN
+F 2 "" H 2780 1260 50  0001 C CNN
+F 3 "" H 2780 1260 50  0001 C CNN
+	1    2780 1260
+	1    0    0    -1
+$EndComp
 NoConn ~ 3000 4010
 $Comp
@@
 Text GLabel 8240 3940 0    50   UnSpc ~ 0
 POS5_IAVG
+$Comp
+L power:GND #PWR?
+U 1 1 5BCB2082
+P 2780 2170
+AR Path="/5BB86F29/5BCB2082" Ref="#PWR?"  Part="1"
+AR Path="/5BB86F26/5BCB2082" Ref="#PWR?"  Part="1"
+F 0 "#PWR?" H 2780 1920 50  0001 C CNN
+F 1 "GND" H 2780 2020 50  0000 C CNN
+F 2 "" H 2780 2170 50  0001 C CNN
+F 3 "" H 2780 2170 50  0001 C CNN
+	1    2780 2170
+	1    0    0    -1
+$EndComp
+Wire Wire Line
+	3000 1760 2780 1760
+Wire Wire Line
+	2780 1760 2780 1640
+Wire Wire Line
+	2780 1760 2780 1870
+Connection ~ 2780 1760
+Wire Wire Line
+	2780 1340 2780 1260
+$Comp
+L Custom_Library:C_Custom C?
+U 1 1 5BCB2091
+P 2780 2020
+F 0 "C?" H 2805 2120 50  0000 L CNN
+F 1 "0.1uF" H 2805 1920 50  0000 L CNN
+F 2 "" H 2818 1870 50  0001 C CNN
+F 3 "" H 2805 2120 50  0001 C CNN
+F 4 "0603" H 2630 2120 50  0000 R CNN "display_footprint"
+F 5 "50V" H 2630 2020 50  0000 R CNN "Voltage"
+F 6 "X7R" H 2630 1920 50  0000 R CNN "Dielectric"
+F 7 "PN" H 3205 2520 60  0001 C CNN "Digi-Key PN"
+	1    2780 2020
+	1    0    0    -1
+$EndComp
+$Comp
+L Custom_Library:R_Custom R?
+U 1 1 5BCB209C
+P 2780 1490
+AR Path="/5BB86F29/5BCB209C" Ref="R?"  Part="1"
+AR Path="/5BB86F26/5BCB209C" Ref="R?"  Part="1"
+F 0 "R?" H 2680 1490 50  0000 R CNN
+F 1 "2" V 2780 1490 50  0000 C CNN
+F 2 "" H 2780 1490 50  0001 C CNN
+F 3 "" H 2780 1490 50  0001 C CNN
+F 4 "PN" H 3080 1890 60  0001 C CNN "Digi-Key PN"
+F 5 "0603" H 2880 1570 50  0000 L CNN "display_footprint"
+F 6 "1%" H 2880 1490 50  0000 L CNN "Tolerance"
+F 7 "1/10W" H 2880 1410 50  0000 L CNN "Wattage"
+	1    2780 1490
+	-1   0    0    -1
+$EndComp
+$Comp
+L power:GND #PWR?
+U 1 1 5BCB2CD0
+P 2780 3420
+AR Path="/5BB86F29/5BCB2CD0" Ref="#PWR?"  Part="1"
+AR Path="/5BB86F26/5BCB2CD0" Ref="#PWR?"  Part="1"
+F 0 "#PWR?" H 2780 3170 50  0001 C CNN
+F 1 "GND" H 2780 3270 50  0000 C CNN
+F 2 "" H 2780 3420 50  0001 C CNN
+F 3 "" H 2780 3420 50  0001 C CNN
+	1    2780 3420
+	1    0    0    -1
+$EndComp
+Wire Wire Line
+	3000 3010 2780 3010
+Wire Wire Line
+	2780 3010 2780 2890
+Wire Wire Line
+	2780 3010 2780 3120
+Connection ~ 2780 3010
+$Comp
+L Custom_Library:C_Custom C?
+U 1 1 5BCB2CDE
+P 2780 3270
+F 0 "C?" H 2805 3370 50  0000 L CNN
+F 1 "0.1uF" H 2805 3170 50  0000 L CNN
+F 2 "" H 2818 3120 50  0001 C CNN
+F 3 "" H 2805 3370 50  0001 C CNN
+F 4 "0603" H 2630 3370 50  0000 R CNN "display_footprint"
+F 5 "50V" H 2630 3270 50  0000 R CNN "Voltage"
+F 6 "X7R" H 2630 3170 50  0000 R CNN "Dielectric"
+F 7 "PN" H 3205 3770 60  0001 C CNN "Digi-Key PN"
+	1    2780 3270
+	1    0    0    -1
+$EndComp
+$Comp
+L Custom_Library:R_Custom R?
+U 1 1 5BCB2CE9
+P 2780 2740
+AR Path="/5BB86F29/5BCB2CE9" Ref="R?"  Part="1"
+AR Path="/5BB86F26/5BCB2CE9" Ref="R?"  Part="1"
+F 0 "R?" H 2680 2740 50  0000 R CNN
+F 1 "2" V 2780 2740 50  0000 C CNN
+F 2 "" H 2780 2740 50  0001 C CNN
+F 3 "" H 2780 2740 50  0001 C CNN
+F 4 "PN" H 3080 3140 60  0001 C CNN "Digi-Key PN"
+F 5 "0603" H 2880 2820 50  0000 L CNN "display_footprint"
+F 6 "1%" H 2880 2740 50  0000 L CNN "Tolerance"
+F 7 "1/10W" H 2880 2660 50  0000 L CNN "Wattage"
+	1    2780 2740
+	-1   0    0    -1
+$EndComp
 $EndSCHEMATC

Commit message: Duplicated master phase, added status LEDs and a few test points
Parts:
- added C? (x3): 0.1uF, symbol Custom_Library:C_Custom
- added D? (x2): Green, symbol Device:LED
- added D?: Red, symbol Device:LED
- added J?: SMOD, symbol Connector_Generic:Conn_02x01
- added J?: RUN, symbol Connector_Generic:Conn_01x03
- added J?: IAVG, symbol Connector_Generic:Conn_02x01
- added R? (x4): 10k, symbol Custom_Library:R_Custom
- added R? (x3): 1k, symbol Custom_Library:R_Custom
- added U? (x2): 74LVC1G06, TO_SOT_Packages_SMD:SOT-353_SC-70-5, symbol Custom_Library:74LVC1G06_Power
- added U?: 74LVC1G17, TO_SOT_Packages_SMD:SOT-353_SC-70-5, symbol Custom_Library:74LVC1G17_Power
- R? (x2): value 2 -> 0
Connections:
- net labels added: POS5_EXTVCC
- net labels removed: ~POS5_DSBL
- wire segments 16 -> 39

Commit message: Assigned some custom footprints
Parts:
- U?: footprint (none) -> Custom Footprints Library:QFN-58-1EP_9x5mm_Pitch0.4mm
Changed lines of the file:
@@
 F 0 "U?" H 2810 1610 50  0000 R CNN
 F 1 "LTC7851UHH" H 2410 5710 50  0000 C CNN
-F 2 "" H -240 4360 50  0001 C CNN
+F 2 "Custom Footprints Library:QFN-58-1EP_9x5mm_Pitch0.4mm" H -240 4360 50  0001 C CNN
 F 3 "http://www.analog.com/media/en/technical-documentation/data-sheets/LTC7851.pdf" H 2410 3660 50  0001 C CNN
 F 4 "LTC7851IUHH#PBF-ND" H 2410 3660 50  0001 C CNN "Digi-Key PN"

Commit message: Annotated schematic
Parts:
- R302: renamed from R?; value 0 -> 2
- gave numbers to parts that had none: 25
Connections:
- net labels added: +5V

Commit message: Cleaned up for ERC
Changed lines of the file:
@@
+	1    0    0    -1
+$EndComp
+Text GLabel 3990 1860 3    50   UnSpc ~ 0
+POS5_EXTVCC
+$Comp
+L power:PWR_FLAG #FLG0101
+U 1 1 5BC417E0
+P 3990 1860
+F 0 "#FLG0101" H 3990 1935 50  0001 C CNN
+F 1 "PWR_FLAG" H 3990 2010 50  0000 C CNN
+F 2 "" H 3990 1860 50  0001 C CNN
+F 3 "~" H 3990 1860 50  0001 C CNN
+	1    3990 1860
 	1    0    0    -1
 $EndComp

Commit message: Added Digi-Key part numbers for all parts
Parts:
- C301, C302, C303, C304, C305: Digi-Key PN PN -> 490-4779-1-ND
- D301: Digi-Key PN (none) -> 160-1447-1-ND
- D302, D303: Digi-Key PN (none) -> 160-1446-1-ND
- R301: Digi-Key PN PN -> 311-0.0GRCT-ND
- R302: Digi-Key PN PN -> RMCF0603FT2R00CT-ND
- R303: Digi-Key PN PN -> P51.1KHCT-ND
- R304, R305, R309, R310: Digi-Key PN PN -> RHM10KADCT-ND
- R306, R307, R308: Digi-Key PN PN -> RHM1.0KDCT-ND
Changed lines of the file:
@@
 F 2 "" H 1780 5780 50  0001 C CNN
 F 3 "" H 1780 5780 50  0001 C CNN
-F 4 "PN" H 2080 6180 60  0001 C CNN "Digi-Key PN"
+F 4 "P51.1KHCT-ND" H 2080 6180 60  0001 C CNN "Digi-Key PN"
 F 5 "0603" H 1880 5860 50  0000 L CNN "display_footprint"
 F 6 "1%" H 1880 5780 50  0000 L CNN "Tolerance"
@@
 F 5 "50V" H 1490 2020 50  0000 R CNN "Voltage"
 F 6 "X7R" H 1490 1920 50  0000 R CNN "Dielectric"
-F 7 "PN" H 2065 2520 60  0001 C CNN "Digi-Key PN"
+F 7 "490-4779-1-ND" H 2065 2520 60  0001 C CNN "Digi-Key PN"
 	1    1640 2020
 	1    0    0    -1
@@
 F 2 "" H 1640 1490 50  0001 C CNN
 F 3 "" H 1640 1490 50  0001 C CNN
-F 4 "PN" H 1940 1890 60  0001 C CNN "Digi-Key PN"
+F 4 "311-0.0GRCT-ND" H 1940 1890 60  0001 C CNN "Digi-Key PN"
 F 5 "0603" H 1740 1570 50  0000 L CNN "display_footprint"
 F 6 "1%" H 1740 1490 50  0000 L CNN "Tolerance"
@@
 F 5 "50V" H 1490 3270 50  0000 R CNN "Voltage"
 F 6 "X7R" H 1490 3170 50  0000 R CNN "Dielectric"
-F 7 "PN" H 2065 3770 60  0001 C CNN "Digi-Key PN"
+F 7 "490-4779-1-ND" H 2065 3770 60  0001 C CNN "Digi-Key PN"
 	1    1640 3270
 	1    0    0    -1
@@
 F 2 "" H 1640 2740 50  0001 C CNN
 F 3 "" H 1640 2740 50  0001 C CNN
-F 4 "PN" H 1940 3140 60  0001 C CNN "Digi-Key PN"
+F 4 "RMCF0603FT2R00CT-ND" H 1940 3140 60  0001 C CNN "Digi-Key PN"
 F 5 "0603" H 1740 2820 50  0000 L CNN "display_footprint"
 F 6 "1%" H 1740 2740 50  0000 L CNN "Tolerance"
@@
 F 5 "1%" H 8800 5470 50  0000 L CNN "Tolerance"
 F 6 "1/10W" H 8800 5390 50  0000 L CNN "Wattage"
-F 7 "PN" H 9020 5870 60  0001 C CNN "Digi-Key PN"
+F 7 "RHM10KADCT-ND" H 9020 5870 60  0001 C CNN "Digi-Key PN"
 	1    8720 5470
 	-1   0    0    -1
@@
 F 5 "1%" H 9010 4270 50  0000 L CNN "Tolerance"
 F 6 "1/10W" H 9010 4190 50  0000 L CNN "Wattage"
-F 7 "PN" H 9230 4670 60  0001 C CNN "Digi-Key PN"
+F 7 "RHM10KADCT-ND" H 9230 4670 60  0001 C CNN "Digi-Key PN"
 	1    8930 4270
 	-1   0    0    -1
@@
 F 5 "1%" H 7120 3260 50  0000 L CNN "Tolerance"
 F 6 "1/10W" H 7120 3180 50  0000 L CNN "Wattage"
-F 7 "PN" H 7340 3660 60  0001 C CNN "Digi-Key PN"
+F 7 "RHM1.0KDCT-ND" H 7340 3660 60  0001 C CNN "Digi-Key PN"
 	1    7040 3260
 	-1   0    0    -1
@@
 F 2 "" H 7040 2960 50  0001 C CNN
 F 3 "~" H 7040 2960 50  0001 C CNN
+F 4 "160-1446-1-ND" H 0   0   50  0001 C CNN "Digi-Key PN"
 	1    7040 2960
 	0    -1   -1   0
@@
 F 5 "1%" H 7120 5320 50  0000 L CNN "Tolerance"
 F 6 "1/10W" H 7120 5240 50  0000 L CNN "Wattage"
-F 7 "PN" H 7340 5720 60  0001 C CNN "Digi-Key PN"
+F 7 "RHM1.0KDCT-ND" H 7340 5720 60  0001 C CNN "Digi-Key PN"
 	1    7040 5320
 	-1   0    0    -1
@@
 F 2 "" H 7040 5020 50  0001 C CNN
 F 3 "~" H 7040 5020 50  0001 C CNN
+F 4 "160-1446-1-ND" H 0   0   50  0001 C CNN "Digi-Key PN"
 	1    7040 5020
 	0    -1   -1   0
@@
 F 5 "1%" H 5850 5270 50  0000 L CNN "Tolerance"
 F 6 "1/10W" H 5850 5190 50  0000 L CNN "Wattage"
-F 7 "PN" H 6070 5670 60  0001 C CNN "Digi-Key PN"
+F 7 "RHM10KADCT-ND" H 6070 5670 60  0001 C CNN "Digi-Key PN"
 	1    5770 5270
 	-1   0    0    -1
@@
 F 5 "50V" H 5780 6020 50  0000 R CNN "Voltage"
 F 6 "X7R" H 5780 5920 50  0000 R CNN "Dielectric"
-F 7 "PN" H 6355 6520 60  0001 C CNN "Digi-Key PN"
+F 7 "490-4779-1-ND" H 6355 6520 60  0001 C CNN "Digi-Key PN"
 	1    5930 6020
 	1    0    0    -1
@@
 F 5 "50V" H 5770 4050 50  0000 R CNN "Voltage"
 F 6 "X7R" H 5770 3950 50  0000 R CNN "Dielectric"
-F 7 "PN" H 6345 4550 60  0001 C CNN "Digi-Key PN"
+F 7 "490-4779-1-ND" H 6345 4550 60  0001 C CNN "Digi-Key PN"
 	1    5920 4050
 	1    0    0    -1
@@
 F 5 "1%" H 7120 1620 50  0000 L CNN "Tolerance"
 F 6 "1/10W" H 7120 1540 50  0000 L CNN "Wattage"
-F 7 "PN" H 7340 2020 60  0001 C CNN "Digi-Key PN"
+F 7 "RHM1.0KDCT-ND" H 7340 2020 60  0001 C CNN "Digi-Key PN"
 	1    7040 1620
 	-1   0    0    -1
@@
 F 2 "" H 7040 1320 50  0001 C CNN
 F 3 "~" H 7040 1320 50  0001 C CNN
+F 4 "160-1447-1-ND" H 0   0   50  0001 C CNN "Digi-Key PN"
 	1    7040 1320
 	0    -1   -1   0
@@
 F 5 "1%" H 5850 1570 50  0000 L CNN "Tolerance"
 F 6 "1/10W" H 5850 1490 50  0000 L CNN "Wattage"
-F 7 "PN" H 6070 1970 60  0001 C CNN "Digi-Key PN"
+F 7 "RHM10KADCT-ND" H 6070 1970 60  0001 C CNN "Digi-Key PN"
 	1    5770 1570
 	-1   0    0    -1
@@
 F 5 "50V" H 5780 2320 50  0000 R CNN "Voltage"
 F 6 "X7R" H 5780 2220 50  0000 R CNN "Dielectric"
-F 7 "PN" H 6355 2820 60  0001 C CNN "Digi-Key PN"
+F 7 "490-4779-1-ND" H 6355 2820 60  0001 C CNN "Digi-Key PN"
 	1    5930 2320
 	1    0    0    -1

Commit message: Assigned footprints
Parts:
- C301, C302, C303, C304, C305: footprint (none) -> Capacitors_SMD:C_0603
- D301, D302, D303: footprint (none) -> LEDs:LED_0603
- J301, J303, J304: footprint (none) -> Pin_Headers:Pin_Header_Straight_1x02_Pitch2.54mm
- J302: footprint (none) -> Pin_Headers:Pin_Header_Straight_1x03_Pitch2.54mm
- R301, R302, R303, R304, R305, R306, R307, R308, R309, R310: footprint (none) -> Resistors_SMD:R_0603
Changed lines of the file:
@@
 F 0 "R303" H 1680 5780 50  0000 R CNN
 F 1 "51.1k" V 1780 5780 40  0000 C CNN
-F 2 "" H 1780 5780 50  0001 C CNN
+F 2 "Resistors_SMD:R_0603" H 1780 5780 50  0001 C CNN
 F 3 "" H 1780 5780 50  0001 C CNN
 F 4 "P51.1KHCT-ND" H 2080 6180 60  0001 C CNN "Digi-Key PN"
@@
 F 0 "J301" H 3300 4390 50  0000 C CNN
 F 1 "CLKOUT" H 3300 4190 50  0000 C CNN
-F 2 "" H 3250 4290 50  0001 C CNN
+F 2 "Pin_Headers:Pin_Header_Straight_1x02_Pitch2.54mm" H 3250 4290 50  0001 C CNN
 F 3 "~" H 3250 4290 50  0001 C CNN
 	1    3250 4290
@@
 F 0 "C301" H 1665 2120 50  0000 L CNN
 F 1 "0.1uF" H 1665 1920 50  0000 L CNN
-F 2 "" H 1678 1870 50  0001 C CNN
+F 2 "Capacitors_SMD:C_0603" H 1678 1870 50  0001 C CNN
 F 3 "" H 1665 2120 50  0001 C CNN
 F 4 "0603" H 1490 2120 50  0000 R CNN "display_footprint"
@@
 F 0 "R301" H 1540 1490 50  0000 R CNN
 F 1 "0" V 1640 1490 50  0000 C CNN
-F 2 "" H 1640 1490 50  0001 C CNN
+F 2 "Resistors_SMD:R_0603" H 1640 1490 50  0001 C CNN
 F 3 "" H 1640 1490 50  0001 C CNN
 F 4 "311-0.0GRCT-ND" H 1940 1890 60  0001 C CNN "Digi-Key PN"
@@
 F 0 "C302" H 1665 3370 50  0000 L CNN
 F 1 "0.1uF" H 1665 3170 50  0000 L CNN
-F 2 "" H 1678 3120 50  0001 C CNN
+F 2 "Capacitors_SMD:C_0603" H 1678 3120 50  0001 C CNN
 F 3 "" H 1665 3370 50  0001 C CNN
 F 4 "0603" H 1490 3370 50  0000 R CNN "display_footprint"
@@
 F 0 "R302" H 1540 2740 50  0000 R CNN
 F 1 "2" V 1640 2740 50  0000 C CNN
-F 2 "" H 1640 2740 50  0001 C CNN
+F 2 "Resistors_SMD:R_0603" H 1640 2740 50  0001 C CNN
 F 3 "" H 1640 2740 50  0001 C CNN
 F 4 "RMCF0603FT2R00CT-ND" H 1940 3140 60  0001 C CNN "Digi-Key PN"
@@
 F 0 "R309" H 8620 5470 50  0000 R CNN
 F 1 "10k" V 8720 5470 50  0000 C CNN
-F 2 "" H 8720 5470 50  0001 C CNN
+F 2 "Resistors_SMD:R_0603" H 8720 5470 50  0001 C CNN
 F 3 "" H 8720 5470 50  0001 C CNN
 F 4 "0603" H 8800 5550 50  0000 L CNN "display_footprint"
@@
 F 0 "J303" H 8770 6070 50  0000 C CNN
 F 1 "SMOD" H 8770 5870 50  0000 C CNN
-F 2 "" H 8720 5970 50  0001 C CNN
+F 2 "Pin_Headers:Pin_Header_Straight_1x02_Pitch2.54mm" H 8720 5970 50  0001 C CNN
 F 3 "~" H 8720 5970 50  0001 C CNN
 	1    8720 5970
@@
 F 0 "J302" H 8260 4070 50  0000 C CNN
 F 1 "RUN" H 8260 3670 50  0000 C CNN
-F 2 "" H 8260 3870 50  0001 C CNN
+F 2 "Pin_Headers:Pin_Header_Straight_1x03_Pitch2.54mm" H 8260 3870 50  0001 C CNN
 F 3 "~" H 8260 3870 50  0001 C CNN
 	1    8260 3870
@@
 F 0 "R310" H 8830 4270 50  0000 R CNN
 F 1 "10k" V 8930 4270 50  0000 C CNN
-F 2 "" H 8930 4270 50  0001 C CNN
+F 2 "Resistors_SMD:R_0603" H 8930 4270 50  0001 C CNN
 F 3 "" H 8930 4270 50  0001 C CNN
 F 4 "0603" H 9010 4350 50  0000 L CNN "display_footprint"
@@
 F 0 "R307" H 6940 3260 50  0000 R CNN
 F 1 "1k" V 7040 3260 50  0000 C CNN
-F 2 "" H 7040 3260 50  0001 C CNN
+F 2 "Resistors_SMD:R_0603" H 7040 3260 50  0001 C CNN
 F 3 "" H 7040 3260 50  0001 C CNN
 F 4 "0603" H 7120 3340 50  0000 L CNN "display_footprint"
@@
 F 0 "D302" H 7040 3060 50  0000 C CNN
 F 1 "Green" H 7040 2860 50  0000 C CNN
-F 2 "" H 7040 2960 50  0001 C CNN
+F 2 "LEDs:LED_0603" H 7040 2960 50  0001 C CNN
 F 3 "~" H 7040 2960 50  0001 C CNN
 F 4 "160-1446-1-ND" H 0   0   50  0001 C CNN "Digi-Key PN"
@@
 F 0 "R308" H 6940 5320 50  0000 R CNN
 F 1 "1k" V 7040 5320 50  0000 C CNN
-F 2 "" H 7040 5320 50  0001 C CNN
+F 2 "Resistors_SMD:R_0603" H 7040 5320 50  0001 C CNN
 F 3 "" H 7040 5320 50  0001 C CNN
 F 4 "0603" H 7120 5400 50  0000 L CNN "display_footprint"
@@
 F 0 "D303" H 7040 5120 50  0000 C CNN
 F 1 "Green" H 7040 4920 50  0000 C CNN
-F 2 "" H 7040 5020 50  0001 C CNN
+F 2 "LEDs:LED_0603" H 7040 5020 50  0001 C CNN
 F 3 "~" H 7040 5020 50  0001 C CNN
 F 4 "160-1446-1-ND" H 0   0   50  0001 C CNN "Digi-Key PN"
@@
 F 0 "R305" H 5670 5270 50  0000 R CNN
 F 1 "10k" V 5770 5270 50  0000 C CNN
-F 2 "" H 5770 5270 50  0001 C CNN
+F 2 "Resistors_SMD:R_0603" H 5770 5270 50  0001 C CNN
 F 3 "" H 5770 5270 50  0001 C CNN
 F 4 "0603" H 5850 5350 50  0000 L CNN "display_footprint"
@@
 F 0 "C305" H 5955 6120 50  0000 L CNN
 F 1 "0.1uF" H 5955 5920 50  0000 L CNN
-F 2 "" H 5968 5870 50  0001 C CNN
+F 2 "Capacitors_SMD:C_0603" H 5968 5870 50  0001 C CNN
 F 3 "" H 5955 6120 50  0001 C CNN
 F 4 "0603" H 5780 6120 50  0000 R CNN "display_footprint"
@@
 F 0 "C303" H 5945 4150 50  0000 L CNN
 F 1 "0.1uF" H 5945 3950 50  0000 L CNN
-F 2 "" H 5958 3900 50  0001 C CNN
+F 2 "Capacitors_SMD:C_0603" H 5958 3900 50  0001 C CNN
 F 3 "" H 5945 4150 50  0001 C CNN
 F 4 "0603" H 5770 4150 50  0000 R CNN "display_footprint"
@@
 F 0 "R306" H 6940 1620 50  0000 R CNN
 F 1 "1k" V 7040 1620 50  0000 C CNN
-F 2 "" H 7040 1620 50  0001 C CNN
+F 2 "Resistors_SMD:R_0603" H 7040 1620 50  0001 C CNN
 F 3 "" H 7040 1620 50  0001 C CNN
 F 4 "0603" H 7120 1700 50  0000 L CNN "display_footprint"
@@
 F 0 "D301" H 7040 1420 50  0000 C CNN
 F 1 "Red" H 7040 1220 50  0000 C CNN
-F 2 "" H 7040 1320 50  0001 C CNN
+F 2 "LEDs:LED_0603" H 7040 1320 50  0001 C CNN
 F 3 "~" H 7040 1320 50  0001 C CNN
 F 4 "160-1447-1-ND" H 0   0   50  0001 C CNN "Digi-Key PN"
@@
 F 0 "R304" H 5670 1570 50  0000 R CNN
 F 1 "10k" V 5770 1570 50  0000 C CNN
-F 2 "" H 5770 1570 50  0001 C CNN
+F 2 "Resistors_SMD:R_0603" H 5770 1570 50  0001 C CNN
 F 3 "" H 5770 1570 50  0001 C CNN
 F 4 "0603" H 5850 1650 50  0000 L CNN "display_footprint"
@@
 F 0 "C304" H 5955 2420 50  0000 L CNN
 F 1 "0.1uF" H 5955 2220 50  0000 L CNN
-F 2 "" H 5968 2170 50  0001 C CNN
+F 2 "Capacitors_SMD:C_0603" H 5968 2170 50  0001 C CNN
 F 3 "" H 5955 2420 50  0001 C CNN
 F 4 "0603" H 5780 2420 50  0000 R CNN "display_footprint"
@@
 F 0 "J304" H 9090 2360 50  0000 C CNN
 F 1 "IAVG" H 9090 2160 50  0000 C CNN
-F 2 "" H 9040 2260 50  0001 C CNN
+F 2 "Pin_Headers:Pin_Header_Straight_1x02_Pitch2.54mm" H 9040 2260 50  0001 C CNN
 F 3 "~" H 9040 2260 50  0001 C CNN
 	1    9040 2260
