File: hdw/LTC7851_Demo/POS5_Phase_1.sch (KiCad schematic (older format))
At the start: 37 parts

Commit message: Added active load sheets
Parts:
- removed C?: C, symbol Custom_Library:C_Custom
- removed R?: R, symbol Custom_Library:R_Custom
- added C?: 0.1uF, symbol Custom_Library:C_Custom
- added R?: 2, symbol Custom_Library:R_Custom
- added R?: 10, symbol Custom_Library:R_Custom
- C?: value C -> 1uF; Dielectric Er -> X7R; Voltage V -> 16V; display_footprint Foot -> 0603
- C?: value C -> 0.1uF; Dielectric Er -> X7R; Voltage V -> 50V; display_footprint Foot -> 0603
- R?: value R -> 2; Tolerance Tol -> 1%; Wattage W -> 1/10W; display_footprint Foot -> 0603
Connections:
- net labels added: +12V, LOOP_TAP
- wire segments 173 -> 175
Changed lines of the file:
@@
 $Descr A 11000 8500
 encoding utf-8
-Sheet 4 13
+Sheet 4 15
 Title ""
 Date ""
@@
 P 3820 1900
 F 0 "C?" H 3845 2000 50  0000 L CNN
-F 1 "C" H 3845 1800 50  0000 L CNN
+F 1 "1uF" H 3845 1800 50  0000 L CNN
 F 2 "" H 3858 1750 50  0001 C CNN
 F 3 "" H 3845 2000 50  0001 C CNN
-F 4 "Foot" H 3670 2000 50  0000 R CNN "display_footprint"
-F 5 "V" H 3670 1900 50  0000 R CNN "Voltage"
-F 6 "Er" H 3670 1800 50  0000 R CNN "Dielectric"
+F 4 "0603" H 3670 2000 50  0000 R CNN "display_footprint"
+F 5 "16V" H 3670 1900 50  0000 R CNN "Voltage"
+F 6 "X7R" H 3670 1800 50  0000 R CNN "Dielectric"
 F 7 "PN" H 4245 2400 60  0001 C CNN "Digi-Key PN"
 	1    3820 1900
-	1    0    0    -1
-$EndComp
-$Comp
-L Custom_Library:R_Custom R?
-U 1 1 5BB8777F
-P 4440 1900
-F 0 "R?" H 4340 1900 50  0000 R CNN
-F 1 "R" V 4440 1900 50  0000 C CNN
-F 2 "" H 4440 1900 50  0001 C CNN
-F 3 "" H 4440 1900 50  0001 C CNN
-F 4 "PN" H 4740 2300 60  0001 C CNN "Digi-Key PN"
-F 5 "Foot" H 4540 1980 50  0000 L CNN "display_footprint"
-F 6 "Tol" H 4540 1900 50  0000 L CNN "Tolerance"
-F 7 "W" H 4540 1820 50  0000 L CNN "Wattage"
-	1    4440 1900
-	1    0    0    -1
-$EndComp
-$Comp
-L Custom_Library:C_Custom C?
-U 1 1 5BB87B44
-P 4440 2430
-F 0 "C?" H 4465 2530 50  0000 L CNN
-F 1 "C" H 4465 2330 50  0000 L CNN
-F 2 "" H 4478 2280 50  0001 C CNN
-F 3 "" H 4465 2530 50  0001 C CNN
-F 4 "Foot" H 4290 2530 50  0000 R CNN "display_footprint"
-F 5 "V" H 4290 2430 50  0000 R CNN "Voltage"
-F 6 "Er" H 4290 2330 50  0000 R CNN "Dielectric"
-F 7 "PN" H 4865 2930 60  0001 C CNN "Digi-Key PN"
-	1    4440 2430
 	1    0    0    -1
 $EndComp
@@
 P 6240 3030
 F 0 "R?" H 6140 3030 50  0000 R CNN
-F 1 "R" V 6240 3030 50  0000 C CNN
+F 1 "2" V 6240 3030 50  0000 C CNN
 F 2 "" H 6240 3030 50  0001 C CNN
 F 3 "" H 6240 3030 50  0001 C CNN
 F 4 "PN" H 6540 3430 60  0001 C CNN "Digi-Key PN"
-F 5 "Foot" H 6340 3110 50  0000 L CNN "display_footprint"
-F 6 "Tol" H 6340 3030 50  0000 L CNN "Tolerance"
-F 7 "W" H 6340 2950 50  0000 L CNN "Wattage"
+F 5 "0603" H 6340 3110 50  0000 L CNN "display_footprint"
+F 6 "1%" H 6340 3030 50  0000 L CNN "Tolerance"
+F 7 "1/10W" H 6340 2950 50  0000 L CNN "Wattage"
 	1    6240 3030
 	-1   0    0    -1
@@
 P 6240 3410
 F 0 "C?" H 6265 3510 50  0000 L CNN
-F 1 "C" H 6265 3310 50  0000 L CNN
+F 1 "0.1uF" H 6265 3310 50  0000 L CNN
 F 2 "" H 6278 3260 50  0001 C CNN
 F 3 "" H 6265 3510 50  0001 C CNN
-F 4 "Foot" H 6090 3510 50  0000 R CNN "display_footprint"
-F 5 "V" H 6090 3410 50  0000 R CNN "Voltage"
-F 6 "Er" H 6090 3310 50  0000 R CNN "Dielectric"
+F 4 "0603" H 6090 3510 50  0000 R CNN "display_footprint"
+F 5 "50V" H 6090 3410 50  0000 R CNN "Voltage"
+F 6 "X7R" H 6090 3310 50  0000 R CNN "Dielectric"
 F 7 "PN" H 6665 3910 60  0001 C CNN "Digi-Key PN"
 	1    6240 3410
@@
 L Custom_Library:R_Custom R?
 U 1 1 5BC4AD64
-P 7200 5280
-F 0 "R?" H 7100 5280 50  0000 R CNN
-F 1 "R" V 7200 5280 50  0000 C CNN
-F 2 "" H 7200 5280 50  0001 C CNN
-F 3 "" H 7200 5280 50  0001 C CNN
-F 4 "PN" H 7500 5680 60  0001 C CNN "Digi-Key PN"
-F 5 "Foot" H 7300 5360 50  0000 L CNN "display_footprint"
-F 6 "Tol" H 7300 5280 50  0000 L CNN "Tolerance"
-F 7 "W" H 7300 5200 50  0000 L CNN "Wattage"
-	1    7200 5280
+P 7200 5470
+F 0 "R?" H 7100 5470 50  0000 R CNN
+F 1 "R" V 7200 5470 50  0000 C CNN
+F 2 "" H 7200 5470 50  0001 C CNN
+F 3 "" H 7200 5470 50  0001 C CNN
+F 4 "PN" H 7500 5870 60  0001 C CNN "Digi-Key PN"
+F 5 "Foot" H 7300 5550 50  0000 L CNN "display_footprint"
+F 6 "Tol" H 7300 5470 50  0000 L CNN "Tolerance"
+F 7 "W" H 7300 5390 50  0000 L CNN "Wattage"
+	1    7200 5470
 	-1   0    0    -1
 $EndComp
@@
 L Custom_Library:R_Custom R?
 U 1 1 5BC4B13D
-P 7200 5750
-F 0 "R?" H 7100 5750 50  0000 R CNN
-F 1 "R" V 7200 5750 50  0000 C CNN
-F 2 "" H 7200 5750 50  0001 C CNN
-F 3 "" H 7200 5750 50  0001 C CNN
-F 4 "PN" H 7500 6150 60  0001 C CNN "Digi-Key PN"
-F 5 "Foot" H 7300 5830 50  0000 L CNN "display_footprint"
-F 6 "Tol" H 7300 5750 50  0000 L CNN "Tolerance"
-F 7 "W" H 7300 5670 50  0000 L CNN "Wattage"
-	1    7200 5750
+P 7200 5940
+F 0 "R?" H 7100 5940 50  0000 R CNN
+F 1 "R" V 7200 5940 50  0000 C CNN
+F 2 "" H 7200 5940 50  0001 C CNN
+F 3 "" H 7200 5940 50  0001 C CNN
+F 4 "PN" H 7500 6340 60  0001 C CNN "Digi-Key PN"
+F 5 "Foot" H 7300 6020 50  0000 L CNN "display_footprint"
+F 6 "Tol" H 7300 5940 50  0000 L CNN "Tolerance"
+F 7 "W" H 7300 5860 50  0000 L CNN "Wattage"
+	1    7200 5940
 	-1   0    0    -1
 $EndComp
-Connection ~ 7200 4540
 $Comp
 L power:GND #PWR?
 U 1 1 5BC4F0D5
-P 7200 6060
-F 0 "#PWR?" H 7200 5810 50  0001 C CNN
-F 1 "GND" H 7200 5910 50  0000 C CNN
-F 2 "" H 7200 6060 50  0001 C CNN
-F 3 "" H 7200 6060 50  0001 C CNN
-	1    7200 6060
-	1    0    0    -1
-$EndComp
-Wire Wire Line
-	7200 6060 7200 5980
-Wire Wire Line
-	7200 5600 7200 5510
+P 7200 6250
+F 0 "#PWR?" H 7200 6000 50  0001 C CNN
+F 1 "GND" H 7200 6100 50  0000 C CNN
+F 2 "" H 7200 6250 50  0001 C CNN
+F 3 "" H 7200 6250 50  0001 C CNN
+	1    7200 6250
+	1    0    0    -1
+$EndComp
+Wire Wire Line
+	7200 6250 7200 6170
+Wire Wire Line
+	7200 5790 7200 5700
 Wire Wire Line
 	4270 4470 4270 5700
-Wire Wire Line
-	4270 5700 6850 5700
-Wire Wire Line
-	7200 4540 7200 5130
-Wire Wire Line
-	6850 5510 7200 5510
-Wire Wire Line
-	6850 5510 6850 5700
-Connection ~ 7200 5510
-Wire Wire Line
-	7200 5510 7200 5430
+Connection ~ 7200 5700
+Wire Wire Line
+	7200 5700 7200 5620
 Wire Wire Line
 	4170 4570 4170 5800
@@
 	4170 5800 6850 5800
 Wire Wire Line
-	6850 5800 6850 5980
-Wire Wire Line
-	6850 5980 7200 5980
-Connection ~ 7200 5980
-Wire Wire Line
-	7200 5980 7200 5900
+	6850 6170 7200 6170
+Connection ~ 7200 6170
+Wire Wire Line
+	7200 6170 7200 6090
 $Comp
 L Custom_Library:R_Custom R?
@@
 	1    0    0    -1
 $EndComp
+$Comp
+L Custom_Library:C_Custom C?
+U 1 1 5BBF5660
+P 4440 2430
+F 0 "C?" H 4465 2530 50  0000 L CNN
+F 1 "0.1uF" H 4465 2330 50  0000 L CNN
+F 2 "" H 4478 2280 50  0001 C CNN
+F 3 "" H 4465 2530 50  0001 C CNN
+F 4 "0603" H 4290 2530 50  0000 R CNN "display_footprint"
+F 5 "50V" H 4290 2430 50  0000 R CNN "Voltage"
+F 6 "X7R" H 4290 2330 50  0000 R CNN "Dielectric"
+F 7 "PN" H 4865 2930 60  0001 C CNN "Digi-Key PN"
+	1    4440 2430
+	1    0    0    -1
+$EndComp
+$Comp
+L Custom_Library:R_Custom R?
+U 1 1 5BBF579B
+P 4440 1900
+F 0 "R?" H 4340 1900 50  0000 R CNN
+F 1 "2" V 4440 1900 50  0000 C CNN
+F 2 "" H 4440 1900 50  0001 C CNN
+F 3 "" H 4440 1900 50  0001 C CNN
+F 4 "PN" H 4740 2300 60  0001 C CNN "Digi-Key PN"
+F 5 "0603" H 4540 1980 50  0000 L CNN "display_footprint"
+F 6 "1%" H 4540 1900 50  0000 L CNN "Tolerance"
+F 7 "1/10W" H 4540 1820 50  0000 L CNN "Wattage"
+	1    4440 1900
+	-1   0    0    -1
+$EndComp
+$Comp
+L power:+12V #PWR?
+U 1 1 5BBF5BBC
+P 8340 1590
+F 0 "#PWR?" H 8340 1440 50  0001 C CNN
+F 1 "+12V" H 8340 1730 50  0000 C CNN
+F 2 "" H 8340 1590 50  0001 C CNN
+F 3 "" H 8340 1590 50  0001 C CNN
+	1    8340 1590
+	1    0    0    -1
+$EndComp
+Wire Wire Line
+	8340 1590 8340 1670
+Connection ~ 8340 1670
+$Comp
+L Custom_Library:R_Custom R?
+U 1 1 5BBFEF87
+P 7200 5090
+F 0 "R?" H 7100 5090 50  0000 R CNN
+F 1 "10" V 7200 5090 50  0000 C CNN
+F 2 "" H 7200 5090 50  0001 C CNN
+F 3 "" H 7200 5090 50  0001 C CNN
+F 4 "PN" H 7500 5490 60  0001 C CNN "Digi-Key PN"
+F 5 "0603" H 7300 5170 50  0000 L CNN "display_footprint"
+F 6 "1%" H 7300 5090 50  0000 L CNN "Tolerance"
+F 7 "1/10W" H 7300 5010 50  0000 L CNN "Wattage"
+	1    7200 5090
+	-1   0    0    -1
+$EndComp
+Wire Wire Line
+	7200 5320 7200 5280
+Connection ~ 7200 4540
+Wire Wire Line
+	4270 5700 7200 5700
+Wire Wire Line
+	6850 5800 6850 6170
+Wire Wire Line
+	7200 4540 7200 4940
+Text GLabel 7280 5280 2    50   UnSpc ~ 0
+LOOP_TAP
+Wire Wire Line
+	7280 5280 7200 5280
+Connection ~ 7200 5280
+Wire Wire Line
+	7200 5280 7200 5240
 $EndSCHEMATC

Commit message: Added component values for all phase 1 components
Parts:
- removed C? (x9): C, symbol Custom_Library:C_Custom
- removed C? (x5): C, symbol Custom_Library:CP_Tant_Custom
- removed R? (x4): R, symbol Custom_Library:R_Custom
- added C?: 1uF, symbol Custom_Library:C_Custom
- added C? (x6): 100uF, symbol Custom_Library:CP_Tant_Custom
- added C?: 100uF, symbol Custom_Library:C_Custom
- added C?: 22uF, symbol Custom_Library:C_Custom
- added C? (x2): 100pF, symbol Custom_Library:C_Custom
- added R?: 13.7k, symbol Custom_Library:R_Custom
- added R?: 10k, symbol Custom_Library:R_Custom
- added R?: 320, symbol Custom_Library:R_Custom
- added R?: 6.04k, symbol Custom_Library:R_Custom
- C?: value C -> 0.22uF; Dielectric Er -> X7R; Voltage V -> 50V; display_footprint Foot -> 0603
- C?: value C -> 22uF; Dielectric Er -> X5R; Digi-Key PN PN -> 445-1436-1-ND; Voltage V -> 25V; display_footprint Foot -> 1210
- C?: value C -> 100uF; Dielectric Er -> X5R; Voltage V -> 10V; display_footprint Foot -> 1210
- C?: value C -> 2200pF; Dielectric Er -> NP0; Voltage V -> 50V; display_footprint Foot -> 0603
- C?: value C -> 100pF; Dielectric Er -> NP0; Voltage V -> 50V; display_footprint Foot -> 0603
- C?: value C -> 3300pF; Dielectric Er -> NP0; Voltage V -> 50V; display_footprint Foot -> 0603
- L?: value L -> 0.47uH; Ampacity A -> 30A; Digi-Key PN (none) -> 541-2595-1-ND; Tolerance Tol -> 20%; display_footprint Foot -> IHLP4040
- R?: value R -> 1.4k; Tolerance Tol -> 1%; Wattage W -> 1/10W; display_footprint Foot -> 0603
- R?: value R -> 100k; Tolerance Tol -> 1%; Wattage W -> 1/10W; display_footprint Foot -> 0603
- R?: value R -> 66.5k; Tolerance Tol -> 1%; Wattage W -> 1/10W; display_footprint Foot -> 0603
Connections:
- wire segments 175 -> 158
Other:
- note added: "Remove bulk caps from onsheet when bringing into project\nAlso remove loop test 10R resistor"

Commit message: Duplicated master phase, added status LEDs and a few test points
Parts:
- added R?: 0, symbol Custom_Library:R_Custom
Connections:
- net labels added: POS5_ISNS1_+, POS5_ISNS1_-, POS5_VSNS1_+, POS5_VSNS1_-
- net labels removed: ~POS5_DSBL
- wire segments 158 -> 155
Other:
- note added: "Remove bulk caps from onsheet when bringing into project\nAlso replace 10R FB resistor with 0R jumper"
- note added: "Route as diff pairs"
- note removed: "Remove bulk caps from onsheet when bringing into project\nAlso remove loop test 10R resistor"

Commit message: Assigned some custom footprints
Parts:
- U?: footprint (none) -> Custom Footprints Library:MLP66-40_6x6mm_Pitch0.5mm
- U?: footprint (none) -> Custom Footprints Library:QFN-58-1EP_9x5mm_Pitch0.4mm
Connections:
- wire segments 155 -> 157
Changed lines of the file:
@@
 F 0 "U?" H 6080 960 50  0000 C CNN
 F 1 "SiC779" H 6080 4660 50  0000 C CNN
-F 2 "" H 4430 3560 50  0001 C CNN
+F 2 "Custom Footprints Library:MLP66-40_6x6mm_Pitch0.5mm" H 4430 3560 50  0001 C CNN
 F 3 "http://www.vishay.com/docs/67538/sic779.pdf" H 6080 2810 50  0001 C CNN
 F 4 "SIC779CD-T1-GE3CT-ND" H 6080 2810 50  0001 C CNN "Digi-Key PN"
@@
 F 0 "U?" H 2910 2160 50  0000 R CNN
 F 1 "LTC7851UHH" H 2510 6260 50  0000 C CNN
-F 2 "" H -140 4910 50  0001 C CNN
+F 2 "Custom Footprints Library:QFN-58-1EP_9x5mm_Pitch0.4mm" H -140 4910 50  0001 C CNN
 F 3 "http://www.analog.com/media/en/technical-documentation/data-sheets/LTC7851.pdf" H 2510 4210 50  0001 C CNN
 F 4 "LTC7851IUHH#PBF-ND" H 2510 4210 50  0001 C CNN "Digi-Key PN"
@@
 Text Notes 3270 3670 0    50   ~ 0
 Route as diff pairs
+Wire Wire Line
+	6730 4110 6810 4110
+Wire Wire Line
+	6810 4110 6810 4010
+Connection ~ 6810 4010
 $EndSCHEMATC

Commit message: Annotated schematic
Parts:
- gave numbers to parts that had none: 36

Commit message: Added Digi-Key part numbers for all parts
Parts:
- C401, C402, C406: Digi-Key PN PN -> 490-4767-1-ND
- C403: Digi-Key PN PN -> 399-9066-1-ND
- C404: Digi-Key PN PN -> 490-4968-1-ND
- C409, C414: Digi-Key PN PN -> 1276-6524-1-ND
- C411, C413: Digi-Key PN PN -> 490-4779-1-ND
- C415: Digi-Key PN PN -> 490-5402-1-ND
- C417: Digi-Key PN PN -> 587-3432-1-ND
- R401: Digi-Key PN PN -> RMCF0603FT66K5CT-ND
- R402: Digi-Key PN PN -> 541-4544-1-ND
- R403: Digi-Key PN PN -> 311-6.04KHRCT-ND
- R404: Digi-Key PN PN -> RHM10KADCT-ND
- R405, R406: Digi-Key PN PN -> RMCF0603FT2R00CT-ND
- R407: Digi-Key PN PN -> P1.40KHCT-ND
- R408: Digi-Key PN PN -> 311-0.0GRCT-ND
- R409: Digi-Key PN PN -> YAG3351CT-ND
- R410: Digi-Key PN PN -> P100KHCT-ND
- R411: Digi-Key PN PN -> P13.7KHCT-ND
Changed lines of the file:
@@
 F 5 "16V" H 4410 1340 50  0000 R CNN "Voltage"
 F 6 "X7R" H 4410 1240 50  0000 R CNN "Dielectric"
-F 7 "PN" H 4985 1840 60  0001 C CNN "Digi-Key PN"
+F 7 "1276-6524-1-ND" H 4985 1840 60  0001 C CNN "Digi-Key PN"
 	1    4560 1340
 	1    0    0    -1
@@
 F 2 "" H 6980 2470 50  0001 C CNN
 F 3 "" H 6980 2470 50  0001 C CNN
-F 4 "PN" H 7280 2870 60  0001 C CNN "Digi-Key PN"
+F 4 "RMCF0603FT2R00CT-ND" H 7280 2870 60  0001 C CNN "Digi-Key PN"
 F 5 "0603" H 7080 2550 50  0000 L CNN "display_footprint"
 F 6 "1%" H 7080 2470 50  0000 L CNN "Tolerance"
@@
 F 5 "50V" H 6830 2850 50  0000 R CNN "Voltage"
 F 6 "X7R" H 6830 2750 50  0000 R CNN "Dielectric"
-F 7 "PN" H 7405 3350 60  0001 C CNN "Digi-Key PN"
+F 7 "490-4779-1-ND" H 7405 3350 60  0001 C CNN "Digi-Key PN"
 	1    6980 2850
 	1    0    0    -1
@@
 F 2 "" H 7190 3770 50  0001 C CNN
 F 3 "" H 7190 3770 50  0001 C CNN
-F 4 "PN" H 7490 4170 60  0001 C CNN "Digi-Key PN"
+F 4 "P1.40KHCT-ND" H 7490 4170 60  0001 C CNN "Digi-Key PN"
 F 5 "0603" H 7290 3850 50  0000 L CNN "display_footprint"
 F 6 "1%" H 7290 3770 50  0000 L CNN "Tolerance"
@@
 F 2 "" H 7478 3890 50  0001 C CNN
 F 3 "" H 7465 4140 50  0001 C CNN
-F 4 "PN" H 7865 4540 60  0001 C CNN "Digi-Key PN"
+F 4 "490-5402-1-ND" H 7865 4540 60  0001 C CNN "Digi-Key PN"
 F 5 "0603" V 7098 4040 50  0000 C CNN "display_footprint"
 F 6 "50V" V 7189 4040 50  0000 C CNN "Voltage"
@@
 F 5 "10V" H 8270 3540 50  0000 R CNN "Voltage"
 F 6 "X5R" H 8270 3440 50  0000 R CNN "Dielectric"
-F 7 "PN" H 8845 4040 60  0001 C CNN "Digi-Key PN"
+F 7 "587-3432-1-ND" H 8845 4040 60  0001 C CNN "Digi-Key PN"
 	1    8420 3540
 	1    0    0    -1
@@
 F 2 "" H 7940 5110 50  0001 C CNN
 F 3 "" H 7940 5110 50  0001 C CNN
-F 4 "PN" H 8240 5510 60  0001 C CNN "Digi-Key PN"
+F 4 "P100KHCT-ND" H 8240 5510 60  0001 C CNN "Digi-Key PN"
 F 5 "0603" H 8040 5190 50  0000 L CNN "display_footprint"
 F 6 "1%" H 8040 5110 50  0000 L CNN "Tolerance"
@@
 F 5 "50V" H 3160 5380 50  0000 R CNN "Voltage"
 F 6 "NP0" H 3160 5280 50  0000 R CNN "Dielectric"
-F 7 "PN" H 3735 5880 60  0001 C CNN "Digi-Key PN"
+F 7 "490-4968-1-ND" H 3735 5880 60  0001 C CNN "Digi-Key PN"
 	1    3310 5380
 	1    0    0    1
@@
 F 5 "50V" H 3700 5610 50  0000 R CNN "Voltage"
 F 6 "NP0" H 3700 5510 50  0000 R CNN "Dielectric"
-F 7 "PN" H 4275 6110 60  0001 C CNN "Digi-Key PN"
+F 7 "490-4767-1-ND" H 4275 6110 60  0001 C CNN "Digi-Key PN"
 	1    3850 5610
 	1    0    0    1
@@
 F 5 "50V" H 3160 4320 50  0000 R CNN "Voltage"
 F 6 "NP0" H 3160 4220 50  0000 R CNN "Dielectric"
-F 7 "PN" H 3735 4820 60  0001 C CNN "Digi-Key PN"
+F 7 "399-9066-1-ND" H 3735 4820 60  0001 C CNN "Digi-Key PN"
 	1    3310 4320
 	1    0    0    -1
@@
 F 2 "" H 1710 6340 50  0001 C CNN
 F 3 "" H 1710 6340 50  0001 C CNN
-F 4 "PN" H 2010 6740 60  0001 C CNN "Digi-Key PN"
+F 4 "RMCF0603FT66K5CT-ND" H 2010 6740 60  0001 C CNN "Digi-Key PN"
 F 5 "0603" H 1810 6420 50  0000 L CNN "display_footprint"
 F 6 "1%" H 1810 6340 50  0000 L CNN "Tolerance"
@@
 F 5 "50V" H 5030 1870 50  0000 R CNN "Voltage"
 F 6 "X7R" H 5030 1770 50  0000 R CNN "Dielectric"
-F 7 "PN" H 5605 2370 60  0001 C CNN "Digi-Key PN"
+F 7 "490-4779-1-ND" H 5605 2370 60  0001 C CNN "Digi-Key PN"
 	1    5180 1870
 	1    0    0    -1
@@
 F 2 "" H 5180 1340 50  0001 C CNN
 F 3 "" H 5180 1340 50  0001 C CNN
-F 4 "PN" H 5480 1740 60  0001 C CNN "Digi-Key PN"
+F 4 "RMCF0603FT2R00CT-ND" H 5480 1740 60  0001 C CNN "Digi-Key PN"
 F 5 "0603" H 5280 1420 50  0000 L CNN "display_footprint"
 F 6 "1%" H 5280 1340 50  0000 L CNN "Tolerance"
@@
 F 2 "" H 7940 4730 50  0001 C CNN
 F 3 "" H 7940 4730 50  0001 C CNN
-F 4 "PN" H 8240 5130 60  0001 C CNN "Digi-Key PN"
+F 4 "YAG3351CT-ND" H 8240 5130 60  0001 C CNN "Digi-Key PN"
 F 5 "0603" H 8040 4810 50  0000 L CNN "display_footprint"
 F 6 "1%" H 8040 4730 50  0000 L CNN "Tolerance"
@@
 F 5 "16V" H 7130 1340 50  0000 R CNN "Voltage"
 F 6 "X7R" H 7130 1240 50  0000 R CNN "Dielectric"
-F 7 "PN" H 7705 1840 60  0001 C CNN "Digi-Key PN"
+F 7 "1276-6524-1-ND" H 7705 1840 60  0001 C CNN "Digi-Key PN"
 	1    7280 1340
 	1    0    0    -1
@@
 F 2 "" H 7940 5580 50  0001 C CNN
 F 3 "" H 7940 5580 50  0001 C CNN
-F 4 "PN" H 8240 5980 60  0001 C CNN "Digi-Key PN"
+F 4 "P13.7KHCT-ND" H 8240 5980 60  0001 C CNN "Digi-Key PN"
 F 5 "0603" H 8040 5660 50  0000 L CNN "display_footprint"
 F 6 "1%" H 8040 5580 50  0000 L CNN "Tolerance"
@@
 F 2 "" H 3850 4620 50  0001 C CNN
 F 3 "" H 3850 4620 50  0001 C CNN
-F 4 "PN" H 4150 5020 60  0001 C CNN "Digi-Key PN"
+F 4 "RHM10KADCT-ND" H 4150 5020 60  0001 C CNN "Digi-Key PN"
 F 5 "0603" H 3950 4700 50  0000 L CNN "display_footprint"
 F 6 "1%" H 3950 4620 50  0000 L CNN "Tolerance"
@@
 F 2 "" H 3310 4780 50  0001 C CNN
 F 3 "" H 3310 4780 50  0001 C CNN
-F 4 "PN" H 3610 5180 60  0001 C CNN "Digi-Key PN"
+F 4 "541-4544-1-ND" H 3610 5180 60  0001 C CNN "Digi-Key PN"
 F 5 "0603" H 3410 4860 50  0000 L CNN "display_footprint"
 F 6 "1%" H 3410 4780 50  0000 L CNN "Tolerance"
@@
 F 2 "" H 3310 5840 50  0001 C CNN
 F 3 "" H 3310 5840 50  0001 C CNN
-F 4 "PN" H 3610 6240 60  0001 C CNN "Digi-Key PN"
+F 4 "311-6.04KHRCT-ND" H 3610 6240 60  0001 C CNN "Digi-Key PN"
 F 5 "0603" H 3410 5920 50  0000 L CNN "display_footprint"
 F 6 "1%" H 3410 5840 50  0000 L CNN "Tolerance"
@@
 F 5 "50V" H 1560 5740 50  0000 R CNN "Voltage"
 F 6 "NP0" H 1560 5640 50  0000 R CNN "Dielectric"
-F 7 "PN" H 2135 6240 60  0001 C CNN "Digi-Key PN"
+F 7 "490-4767-1-ND" H 2135 6240 60  0001 C CNN "Digi-Key PN"
 	1    1710 5740
 	-1   0    0    -1
@@
 F 5 "50V" H 1560 5140 50  0000 R CNN "Voltage"
 F 6 "NP0" H 1560 5040 50  0000 R CNN "Dielectric"
-F 7 "PN" H 2135 5640 60  0001 C CNN "Digi-Key PN"
+F 7 "490-4767-1-ND" H 2135 5640 60  0001 C CNN "Digi-Key PN"
 	1    1710 5140
 	-1   0    0    -1
@@
 F 5 "1%" V 7474 5810 50  0000 C CNN "Tolerance"
 F 6 "1/10W" V 7565 5810 50  0000 C CNN "Wattage"
-F 7 "PN" H 7980 6210 60  0001 C CNN "Digi-Key PN"
+F 7 "311-0.0GRCT-ND" H 7980 6210 60  0001 C CNN "Digi-Key PN"
 	1    7680 5810
 	0    1    -1   0
