File: hdw/LTC7851_Demo/POS5_Phase_1.sch (KiCad schematic (older format))
At the start: 36 parts, among them U301 LTC7851UHH, U401 SiC779

Commit message: More routing, removed GL ang GH phase test points
Parts:
- removed TP401, TP402: TP, Measurement_Points:Measurement_Point_Round-SMD-Pad_Small, symbol Custom_Library:TP
Connections:
- no-connect marks 0 -> 2
Changed lines of the file:
@@
 ~POS5_THDN
-$Comp
-L Custom_Library:TP TP401
-U 1 1 5BB96CFD
-P 5430 2810
-F 0 "TP401" V 5430 2960 50  0000 L CNN
-F 1 "TP" H 5430 2960 50  0001 C CNN
-F 2 "Measurement_Points:Measurement_Point_Round-SMD-Pad_Small" H 5430 2810 60  0001 C CNN
-F 3 "" H 5430 2810 60  0000 C CNN
-	1    5430 2810
-	0    -1   -1   0
-$EndComp
-$Comp
-L Custom_Library:TP TP402
-U 1 1 5BB96F26
-P 5430 2910
-F 0 "TP402" V 5430 3060 50  0000 L CNN
-F 1 "TP" H 5430 3060 50  0001 C CNN
-F 2 "Measurement_Points:Measurement_Point_Round-SMD-Pad_Small" H 5430 2910 60  0001 C CNN
-F 3 "" H 5430 2910 60  0000 C CNN
-	1    5430 2910
-	0    -1   -1   0
-$EndComp
 $Comp
 L power:GND #PWR0418
@@
 Text Notes 540  690  0    100  ~ 20
 +5V Phase 1
+NoConn ~ 5430 2810
+NoConn ~ 5430 2910
 $EndSCHEMATC

Commit message: Finished ROUTING (for the most part)
Connections:
- net labels removed: POS5_SMOD
- no-connect marks 2 -> 3
Changed lines of the file:
@@
 Wire Wire Line
 	6810 1710 6810 1810
-Text GLabel 5430 3110 0    50   Input ~ 0
-POS5_SMOD
 $Comp
 L Custom_Library:R_Custom R406
@@
 	3850 5460 3850 5110
 Connection ~ 3850 5110
-Text GLabel 5430 2510 0    50   Input ~ 0
-POS5_RUN
 Wire Wire Line
 	7940 5730 7940 5810
@@
 NoConn ~ 5430 2810
 NoConn ~ 5430 2910
+NoConn ~ 5430 3110
+$Comp
+L Custom_Library:+5.5V_MNG #PWR?
+U 1 1 5BCCA9E9
+P 5430 2510
+F 0 "#PWR?" H 5430 2360 50  0001 C CNN
+F 1 "+5.5V_MNG" V 5430 2650 50  0000 L CNN
+F 2 "" H 5430 2510 50  0001 C CNN
+F 3 "" H 5430 2510 50  0001 C CNN
+	1    5430 2510
+	0    -1   -1   0
+$EndComp
 $EndSCHEMATC

Commit message: Added a few connectors and cleaned up some routing
Other:
- note removed: "Remove bulk caps from onsheet when bringing into project\nAlso replace 10R FB resistor with 0R jumper"
Changed lines of the file:
@@
 	1    0    0    -1
 $EndComp
-Text Notes 3330 6760 0    50   ~ 0
-Remove bulk caps from onsheet when bringing into project\nAlso replace 10R FB resistor with 0R jumper
 $Comp
 L Custom_Library:C_Custom C418
@@
 NoConn ~ 5430 3110
 $Comp
-L Custom_Library:+5.5V_MNG #PWR?
+L Custom_Library:+5.5V_MNG #PWR0101
 U 1 1 5BCCA9E9
 P 5430 2510
-F 0 "#PWR?" H 5430 2360 50  0001 C CNN
+F 0 "#PWR0101" H 5430 2360 50  0001 C CNN
 F 1 "+5.5V_MNG" V 5430 2650 50  0000 L CNN
 F 2 "" H 5430 2510 50  0001 C CNN

Commit message: Substantial wiring and layout changes
Parts:
- added R412, R413, R414: 0, Resistors_SMD:R_0402, symbol Custom_Library:R_Custom
- C401, C402, C406: footprint Capacitors_SMD:C_0603 -> Capacitors_SMD:C_0402; Dielectric NP0 -> X7R; Digi-Key PN 490-4767-1-ND -> 478-1089-1-ND; display_footprint 0603 -> 0402
- C403: footprint Capacitors_SMD:C_0603 -> Capacitors_SMD:C_0402; Dielectric NP0 -> X7R; Digi-Key PN 399-9066-1-ND -> 478-5132-1-ND; display_footprint 0603 -> 0402
- C404: footprint Capacitors_SMD:C_0603 -> Capacitors_SMD:C_0402; Dielectric NP0 -> X7R; Digi-Key PN 490-4968-1-ND -> 478-1105-1-ND; display_footprint 0603 -> 0402
- C415: footprint Capacitors_SMD:C_0603 -> Capacitors_SMD:C_0402; Dielectric X7R -> X5R; Digi-Key PN 490-5402-1-ND -> 1276-1049-1-ND; Voltage 50V -> 10V; display_footprint 0603 -> 0402
- R401: footprint Resistors_SMD:R_0603 -> Resistors_SMD:R_0402; Digi-Key PN RMCF0603FT66K5CT-ND -> RMCF0402FT66K5CT-ND; Wattage 1/10W -> 1/16W; display_footprint 0603 -> 0402
- R402: value 320 -> 324; footprint Resistors_SMD:R_0603 -> Resistors_SMD:R_0402; Digi-Key PN 541-4544-1-ND -> YAG3118CT-ND; Wattage 1/10W -> 1/16W; display_footprint 0603 -> 0402
- R403: footprint Resistors_SMD:R_0603 -> Resistors_SMD:R_0402; Digi-Key PN 311-6.04KHRCT-ND -> RMCF0402FT6K04CT-ND; Wattage 1/10W -> 1/16W; display_footprint 0603 -> 0402
- R404: footprint Resistors_SMD:R_0603 -> Resistors_SMD:R_0402; Digi-Key PN RHM10KADCT-ND -> 311-10.0KLRCT-ND; Wattage 1/10W -> 1/16W; display_footprint 0603 -> 0402
- R407: footprint Resistors_SMD:R_0603 -> Resistors_SMD:R_0402; Digi-Key PN P1.40KHCT-ND -> RMCF0402FT1K40CT-ND; Wattage 1/10W -> 1/16W; display_footprint 0603 -> 0402
- R408: footprint Resistors_SMD:R_0603 -> Resistors_SMD:R_0402; Digi-Key PN 311-0.0GRCT-ND -> RMCF0402ZT0R00CT-ND; Wattage 1/10W -> 1/16W; display_footprint 0603 -> 0402
- R409: footprint Resistors_SMD:R_0603 -> Resistors_SMD:R_0402; Digi-Key PN YAG3351CT-ND -> 311-10.0LRCT-ND; Wattage 1/10W -> 1/16W; display_footprint 0603 -> 0402
- R410: footprint Resistors_SMD:R_0603 -> Resistors_SMD:R_0402; Digi-Key PN P100KHCT-ND -> 311-100KLRCT-ND; Wattage 1/10W -> 1/16W; display_footprint 0603 -> 0402
- R411: footprint Resistors_SMD:R_0603 -> Resistors_SMD:R_0402; Digi-Key PN P13.7KHCT-ND -> 311-13.7KLRCT-ND; Wattage 1/10W -> 1/16W; display_footprint 0603 -> 0402
Connections:
- net labels added: POS5_VSNSO1_+, POS5_VSNSO1_-
- net labels removed: POS5_VSNS1_+, POS5_VSNS1_-
- wire segments 157 -> 166
