File: hdw/LTC7851_Demo/Power_Input.sch (KiCad schematic (older format))
At the start: 0 parts

Commit message: Added LDO for VCC input, cleaned some stuff up
Parts:
- added C?: 0.1uF, symbol LED_Display_Local_Library:C_Custom
- added C?: 10nF, symbol LED_Display_Local_Library:C_Custom
- added C?: 1nF, symbol LED_Display_Local_Library:C_Custom
- added C?: C, symbol Custom_Library:C_Custom
- added C? (x3): 100uF, symbol LED_Display_Local_Library:CP_Tant_Custom
- added F?: Fuse, symbol Device:Fuse
- added J? (x3): +12VIN, symbol Connector:Screw_Terminal_01x01
- added J? (x3): GNDIN, symbol Connector:Screw_Terminal_01x01
- added Q? (x2): Q_DUAL_NMOS_G1S2G2D2S1D1, symbol Device:Q_DUAL_NMOS_G1S2G2D2S1D1
- added R? (x5): R, symbol Custom_Library:R_Custom
- added R? (x2): 10, symbol Custom_Library:R_Custom
- added R?: 10k, symbol Custom_Library:R_Custom
- added TP? (x2): TP, symbol Custom_Library:TP
- added U?: LTC4365DDB, Package_DFN_QFN:DFN-8-1EP_2x3mm_P0.5mm_EP0.61x2.2mm, symbol LED_Display_Local_Library:LTC4365DDB
Connections:
- net labels added: +12V, +12Vin, GND, POS12_PGOOD
- wire segments 0 -> 73
Other:
- note added: "SELECT NMOS"
