File: hdw/LTC7851_Demo/Power_Input.sch (KiCad schematic (older format))
At the start: 27 parts

Commit message: Added active load sheets
Connections:
- net labels added: +5.5V_MNG
Changed lines of the file:
@@
 $Descr A 11000 8500
 encoding utf-8
-Sheet 2 13
+Sheet 2 15
 Title ""
 Date ""
@@
 Wire Wire Line
 	2440 4070 2440 4420
+$Comp
+L Custom_Library:+5.5V_MNG #PWR?
+U 1 1 5BBEC090
+P 6050 4260
+F 0 "#PWR?" H 6050 4110 50  0001 C CNN
+F 1 "+5.5V_MNG" H 6050 4400 50  0000 C CNN
+F 2 "" H 6050 4260 50  0001 C CNN
+F 3 "" H 6050 4260 50  0001 C CNN
+	1    6050 4260
+	1    0    0    -1
+$EndComp
 $EndSCHEMATC

Commit message: Filled in power input page
Parts:
- removed C?: C, symbol Custom_Library:C_Custom
- removed Q? (x2): Q_DUAL_NMOS_G1S2G2D2S1D1, symbol Device:Q_DUAL_NMOS_G1S2G2D2S1D1
- added C?: 10nF, symbol LED_Display_Local_Library:C_Custom
- added D?: 24V, Diodes_SMD:D_SMA, symbol Device:D_TVS_ALT
- added F?: 25A, Fuse_Holders_and_Fuses:Fuse_SMD1206_Reflow, symbol Device:Fuse
- added Q? (x2): BSC123N10LSGATMA1, Package_TO_SOT_SMD:TDSON-8-1, symbol Transistor_FET:BSC123N10LSG
- F?: value Fuse -> 25A; footprint (none) -> Fuse_Holders_and_Fuses:Fuse_SMD1206_Reflow
- R?: value R -> 6M
- R?: value R -> 86.6k
- R?: value R -> 243k
- R?: value R -> 100k
- R?: value R -> 5.1k
Connections:
- wire segments 73 -> 81
Other:
- note removed: "SELECT NMOS"

Commit message: Assigned some custom footprints
Parts:
- added C?: 0.1uF, symbol Custom_Library:C_Custom
- added D?: Green, symbol Device:LED
- added R?: 1k, symbol Custom_Library:R_Custom
- added U?: 74LVC1G06, TO_SOT_Packages_SMD:SOT-353_SC-70-5, symbol Custom_Library:74LVC1G06_Power
- J? (x6): footprint (none) -> Custom Footprints Library:Keystone_8191
Connections:
- wire segments 81 -> 83
Changed lines of the file:
@@
 $EndComp
 Wire Wire Line
-	5360 3590 5360 3510
+	5360 3590 5360 3490
 Wire Wire Line
 	5360 3110 5070 3110
@@
 	5360 3110 5640 3110
 Connection ~ 5360 3110
-Connection ~ 5360 3510
-Wire Wire Line
-	5360 3510 5360 3110
+Connection ~ 5360 3490
+Wire Wire Line
+	5360 3490 5360 3110
 $Comp
 L power:GND #PWR?
@@
 F 0 "J?" H 1600 2820 50  0000 C CNN
 F 1 "+12VIN" H 1600 2620 50  0000 C CNN
-F 2 "" H 1600 2720 50  0001 C CNN
+F 2 "Custom Footprints Library:Keystone_8191" H 1600 2720 50  0001 C CNN
 F 3 "~" H 1600 2720 50  0001 C CNN
 	1    1600 2720
@@
 F 0 "J?" H 1600 4520 50  0000 C CNN
 F 1 "GNDIN" H 1600 4320 50  0000 C CNN
-F 2 "" H 1600 4420 50  0001 C CNN
+F 2 "Custom Footprints Library:Keystone_8191" H 1600 4420 50  0001 C CNN
 F 3 "~" H 1600 4420 50  0001 C CNN
 	1    1600 4420
@@
 Connection ~ 7750 2720
 Wire Wire Line
-	7000 3870 7000 3510
-Wire Wire Line
-	5360 3510 7000 3510
+	7000 3870 7000 3490
+Wire Wire Line
+	5360 3490 7000 3490
 $Comp
 L Custom_Library:R_Custom R?
@@
 F 0 "J?" H 1600 3170 50  0000 C CNN
 F 1 "+12VIN" H 1600 2970 50  0000 C CNN
-F 2 "" H 1600 3070 50  0001 C CNN
+F 2 "Custom Footprints Library:Keystone_8191" H 1600 3070 50  0001 C CNN
 F 3 "~" H 1600 3070 50  0001 C CNN
 	1    1600 3070
@@
 F 0 "J?" H 1600 3520 50  0000 C CNN
 F 1 "+12VIN" H 1600 3320 50  0000 C CNN
-F 2 "" H 1600 3420 50  0001 C CNN
+F 2 "Custom Footprints Library:Keystone_8191" H 1600 3420 50  0001 C CNN
 F 3 "~" H 1600 3420 50  0001 C CNN
 	1    1600 3420
@@
 F 0 "J?" H 1600 4170 50  0000 C CNN
 F 1 "GNDIN" H 1600 3970 50  0000 C CNN
-F 2 "" H 1600 4070 50  0001 C CNN
+F 2 "Custom Footprints Library:Keystone_8191" H 1600 4070 50  0001 C CNN
 F 3 "~" H 1600 4070 50  0001 C CNN
 	1    1600 4070
@@
 F 0 "J?" H 1600 3820 50  0000 C CNN
 F 1 "GNDIN" H 1600 3620 50  0000 C CNN
-F 2 "" H 1600 3720 50  0001 C CNN
+F 2 "Custom Footprints Library:Keystone_8191" H 1600 3720 50  0001 C CNN
 F 3 "~" H 1600 3720 50  0001 C CNN
 	1    1600 3720
@@
 	1    0    0    -1
 $EndComp
+$Comp
+L Custom_Library:74LVC1G06_Power U?
+U 1 1 5BC2A9C5
+P 8340 5140
+AR Path="/5BB86F26/5BC2A9C5" Ref="U?"  Part="1"
+AR Path="/5BB86F23/5BC2A9C5" Ref="U?"  Part="1"
+F 0 "U?" H 8440 5290 50  0000 L CNN
+F 1 "74LVC1G06" H 8440 5040 50  0000 L CNN
+F 2 "TO_SOT_Packages_SMD:SOT-353_SC-70-5" H 8340 5190 50  0001 C CNN
+F 3 "http://www.ti.com/lit/ds/symlink/sn74lvc1g06.pdf" H 8340 5140 50  0001 C CNN
+F 4 "296-8484-1-ND" H 8340 5140 50  0001 C CNN "Digi-Key PN"
+	1    8340 5140
+	1    0    0    -1
+$EndComp
+$Comp
+L Custom_Library:+5.5V_MNG #PWR?
+U 1 1 5BC2A9CC
+P 8340 5040
+F 0 "#PWR?" H 8340 4890 50  0001 C CNN
+F 1 "+5.5V_MNG" H 8340 5180 50  0000 C CNN
+F 2 "" H 8340 5040 50  0001 C CNN
+F 3 "" H 8340 5040 50  0001 C CNN
+	1    8340 5040
+	1    0    0    -1
+$EndComp
+$Comp
+L power:GND #PWR?
+U 1 1 5BC2A9D2
+P 8340 5240
+F 0 "#PWR?" H 8340 4990 50  0001 C CNN
+F 1 "GND" H 8340 5090 50  0000 C CNN
+F 2 "" H 8340 5240 50  0001 C CNN
+F 3 "" H 8340 5240 50  0001 C CNN
+	1    8340 5240
+	1    0    0    -1
+$EndComp
+$Comp
+L Custom_Library:R_Custom R?
+U 1 1 5BC2A9DC
+P 9050 4840
+AR Path="/5BB2595E/5BC2A9DC" Ref="R?"  Part="1"
+AR Path="/5BAAE0FA/5BC2A9DC" Ref="R?"  Part="1"
+AR Path="/5BB86F23/5BC2A9DC" Ref="R?"  Part="1"
+AR Path="/5BB86F26/5BC2A9DC" Ref="R?"  Part="1"
+F 0 "R?" H 8950 4840 50  0000 R CNN
+F 1 "1k" V 9050 4840 50  0000 C CNN
+F 2 "" H 9050 4840 50  0001 C CNN
+F 3 "" H 9050 4840 50  0001 C CNN
+F 4 "0603" H 9130 4920 50  0000 L CNN "display_footprint"
+F 5 "1%" H 9130 4840 50  0000 L CNN "Tolerance"
+F 6 "1/10W" H 9130 4760 50  0000 L CNN "Wattage"
+F 7 "PN" H 9350 5240 60  0001 C CNN "Digi-Key PN"
+	1    9050 4840
+	-1   0    0    -1
+$EndComp
+Wire Wire Line
+	9050 4990 9050 5140
+Wire Wire Line
+	9050 5140 8590 5140
+$Comp
+L Device:LED D?
+U 1 1 5BC2A9E5
+P 9050 4540
+F 0 "D?" H 9050 4640 50  0000 C CNN
+F 1 "Green" H 9050 4440 50  0000 C CNN
+F 2 "" H 9050 4540 50  0001 C CNN
+F 3 "~" H 9050 4540 50  0001 C CNN
+	1    9050 4540
+	0    -1   -1   0
+$EndComp
+$Comp
+L Custom_Library:+5.5V_MNG #PWR?
+U 1 1 5BC2A9EC
+P 9050 4390
+F 0 "#PWR?" H 9050 4240 50  0001 C CNN
+F 1 "+5.5V_MNG" H 9050 4530 50  0000 C CNN
+F 2 "" H 9050 4390 50  0001 C CNN
+F 3 "" H 9050 4390 50  0001 C CNN
+	1    9050 4390
+	1    0    0    -1
+$EndComp
+$Comp
+L Custom_Library:C_Custom C?
+U 1 1 5BC2A9F7
+P 7940 5540
+F 0 "C?" H 7965 5640 50  0000 L CNN
+F 1 "0.1uF" H 7965 5440 50  0000 L CNN
+F 2 "" H 7978 5390 50  0001 C CNN
+F 3 "" H 7965 5640 50  0001 C CNN
+F 4 "0603" H 7790 5640 50  0000 R CNN "display_footprint"
+F 5 "50V" H 7790 5540 50  0000 R CNN "Voltage"
+F 6 "X7R" H 7790 5440 50  0000 R CNN "Dielectric"
+F 7 "PN" H 8365 6040 60  0001 C CNN "Digi-Key PN"
+	1    7940 5540
+	1    0    0    -1
+$EndComp
+$Comp
+L Custom_Library:+5.5V_MNG #PWR?
+U 1 1 5BC2A9FE
+P 7940 5390
+F 0 "#PWR?" H 7940 5240 50  0001 C CNN
+F 1 "+5.5V_MNG" H 7940 5530 50  0000 C CNN
+F 2 "" H 7940 5390 50  0001 C CNN
+F 3 "" H 7940 5390 50  0001 C CNN
+	1    7940 5390
+	1    0    0    -1
+$EndComp
+$Comp
+L power:GND #PWR?
+U 1 1 5BC2AA04
+P 7940 5690
+F 0 "#PWR?" H 7940 5440 50  0001 C CNN
+F 1 "GND" H 7940 5540 50  0000 C CNN
+F 2 "" H 7940 5690 50  0001 C CNN
+F 3 "" H 7940 5690 50  0001 C CNN
+	1    7940 5690
+	1    0    0    -1
+$EndComp
+Text GLabel 8040 5140 0    50   Input ~ 0
+POS12_PGOOD
 $EndSCHEMATC

Commit message: Annotated schematic
Parts:
- gave numbers to parts that had none: 33

Commit message: Changed cap voltage rating
Parts:
- C201: Voltage 25V -> 50V
Changed lines of the file:
@@
 F 3 "" H 5175 6370 50  0001 C CNN
 F 4 "0603" H 5000 6370 50  0000 R CNN "display_footprint"
-F 5 "25V" H 5000 6270 50  0000 R CNN "Voltage"
+F 5 "50V" H 5000 6270 50  0000 R CNN "Voltage"
 F 6 "X7R" H 5000 6170 50  0000 R CNN "Dielectric"
 F 7 "PN" H 5575 6770 60  0001 C CNN "Digi-Key PN"

Commit message: Added Digi-Key part numbers for all parts
Parts:
- C201, C207: Digi-Key PN PN -> 490-4779-1-ND
- C202, C205: Digi-Key PN PN -> 1276-1921-1-ND; Voltage 25V -> 50V
- C203: Digi-Key PN PN -> 311-1080-1-ND; Voltage 25V -> 50V
- D202: Digi-Key PN (none) -> 160-1446-1-ND
- F201, F202: Digi-Key PN (none) -> 507-1946-1-ND
- J201, J202, J203, J204, J205, J206: Digi-Key PN (none) -> 36-8191-ND
- R201: value 6M -> 6.04M; Digi-Key PN PN -> 541-6.04MHCT-ND
- R202: Digi-Key PN PN -> 311-86.6KHRCT-ND
- R203: Digi-Key PN PN -> 541-243KHCT-ND
- R204: Digi-Key PN PN -> P100KHCT-ND
- R205, R206: Digi-Key PN PN -> YAG3351CT-ND
- R207: Digi-Key PN PN -> RHM10KADCT-ND
- R208: Digi-Key PN PN -> RMCF0603FT5K10CT-ND
- R209: Digi-Key PN PN -> RHM1.0KDCT-ND
Changed lines of the file:
@@
 AR Path="/5BB86F23/5BB576E9" Ref="R201"  Part="1"
 F 0 "R201" H 2740 4530 50  0000 R CNN
-F 1 "6M" V 2840 4530 50  0000 C CNN
+F 1 "6.04M" V 2840 4530 50  0000 C CNN
 F 2 "" H 2840 4530 50  0001 C CNN
 F 3 "" H 2840 4530 50  0001 C CNN
@@
 F 5 "1%" H 2920 4530 50  0000 L CNN "Tolerance"
 F 6 "1/10W" H 2920 4450 50  0000 L CNN "Wattage"
-F 7 "PN" H 3140 4930 60  0001 C CNN "Digi-Key PN"
+F 7 "541-6.04MHCT-ND" H 3140 4930 60  0001 C CNN "Digi-Key PN"
 	1    2840 4530
 	1    0    0    -1
@@
 F 5 "50V" H 5000 6270 50  0000 R CNN "Voltage"
 F 6 "X7R" H 5000 6170 50  0000 R CNN "Dielectric"
-F 7 "PN" H 5575 6770 60  0001 C CNN "Digi-Key PN"
+F 7 "490-4779-1-ND" H 5575 6770 60  0001 C CNN "Digi-Key PN"
 	1    5150 6270
 	1    0    0    -1
@@
 F 3 "" H 5475 6370 50  0001 C CNN
 F 4 "0603" H 5300 6370 50  0001 R CNN "display_footprint"
-F 5 "25V" H 5300 6270 50  0001 R CNN "Voltage"
+F 5 "50V" H 5300 6270 50  0001 R CNN "Voltage"
 F 6 "X7R" H 5300 6170 50  0001 R CNN "Dielectric"
-F 7 "PN" H 5875 6770 60  0001 C CNN "Digi-Key PN"
+F 7 "1276-1921-1-ND" H 5875 6770 60  0001 C CNN "Digi-Key PN"
 	1    5450 6270
 	1    0    0    -1
@@
 F 3 "" H 5775 6370 50  0001 C CNN
 F 4 "0603" H 5600 6370 50  0001 R CNN "display_footprint"
-F 5 "25V" H 5600 6270 50  0001 R CNN "Voltage"
+F 5 "50V" H 5600 6270 50  0001 R CNN "Voltage"
 F 6 "X7R" H 5600 6170 50  0001 R CNN "Dielectric"
-F 7 "PN" H 6175 6770 60  0001 C CNN "Digi-Key PN"
+F 7 "311-1080-1-ND" H 6175 6770 60  0001 C CNN "Digi-Key PN"
 	1    5750 6270
 	1    0    0    -1
@@
 F 5 "1%" H 2920 5060 50  0000 L CNN "Tolerance"
 F 6 "1/10W" H 2920 4980 50  0000 L CNN "Wattage"
-F 7 "PN" H 3140 5460 60  0001 C CNN "Digi-Key PN"
+F 7 "311-86.6KHRCT-ND" H 3140 5460 60  0001 C CNN "Digi-Key PN"
 	1    2840 5060
 	1    0    0    -1
@@
 F 5 "1%" H 2920 5560 50  0000 L CNN "Tolerance"
 F 6 "1/10W" H 2920 5480 50  0000 L CNN "Wattage"
-F 7 "PN" H 3140 5960 60  0001 C CNN "Digi-Key PN"
+F 7 "541-243KHCT-ND" H 3140 5960 60  0001 C CNN "Digi-Key PN"
 	1    2840 5560
 	1    0    0    -1
@@
 F 5 "1%" H 3450 4040 50  0000 L CNN "Tolerance"
 F 6 "1/10W" H 3450 3960 50  0000 L CNN "Wattage"
-F 7 "PN" H 3670 4440 60  0001 C CNN "Digi-Key PN"
+F 7 "P100KHCT-ND" H 3670 4440 60  0001 C CNN "Digi-Key PN"
 	1    3370 4040
 	1    0    0    -1
@@
 F 5 "1%" V 5120 3110 50  0000 C CNN "Tolerance"
 F 6 "1/10W" V 5220 3110 50  0000 C CNN "Wattage"
-F 7 "PN" H 5220 3510 60  0001 C CNN "Digi-Key PN"
+F 7 "YAG3351CT-ND" H 5220 3510 60  0001 C CNN "Digi-Key PN"
 	1    4920 3110
 	0    1    1    0
@@
 F 5 "1%" V 5990 3110 50  0000 C CNN "Tolerance"
 F 6 "1/10W" V 6090 3110 50  0000 C CNN "Wattage"
-F 7 "PN" H 6090 3510 60  0001 C CNN "Digi-Key PN"
+F 7 "YAG3351CT-ND" H 6090 3510 60  0001 C CNN "Digi-Key PN"
 	1    5790 3110
 	0    1    1    0
@@
 F 5 "1%" H 7080 4020 50  0000 L CNN "Tolerance"
 F 6 "1/10W" H 7080 3940 50  0000 L CNN "Wattage"
-F 7 "PN" H 7300 4420 60  0001 C CNN "Digi-Key PN"
+F 7 "RMCF0603FT5K10CT-ND" H 7300 4420 60  0001 C CNN "Digi-Key PN"
 	1    7000 4020
 	1    0    0    -1
@@
 F 2 "Fuse_Holders_and_Fuses:Fuse_SMD1206_Reflow" V 2250 2720 50  0001 C CNN
 F 3 "~" H 2320 2720 50  0001 C CNN
+F 4 "507-1946-1-ND" H 0   0   50  0001 C CNN "Digi-Key PN"
 	1    2320 2720
 	0    1    1    0
@@
 F 2 "Custom Footprints Library:Keystone_8191" H 1600 2720 50  0001 C CNN
 F 3 "~" H 1600 2720 50  0001 C CNN
+F 4 "36-8191-ND" H 0   0   50  0001 C CNN "Digi-Key PN"
 	1    1600 2720
 	-1   0    0    -1
@@
 F 2 "Custom Footprints Library:Keystone_8191" H 1600 4420 50  0001 C CNN
 F 3 "~" H 1600 4420 50  0001 C CNN
+F 4 "36-8191-ND" H 0   0   50  0001 C CNN "Digi-Key PN"
 	1    1600 4420
 	-1   0    0    -1
@@
 F 5 "1%" H 6130 4410 50  0000 L CNN "Tolerance"
 F 6 "1/10W" H 6130 4330 50  0000 L CNN "Wattage"
-F 7 "PN" H 6350 4810 60  0001 C CNN "Digi-Key PN"
+F 7 "RHM10KADCT-ND" H 6350 4810 60  0001 C CNN "Digi-Key PN"
 	1    6050 4410
 	-1   0    0    -1
@@
 F 2 "Custom Footprints Library:Keystone_8191" H 1600 3070 50  0001 C CNN
 F 3 "~" H 1600 3070 50  0001 C CNN
+F 4 "36-8191-ND" H 0   0   50  0001 C CNN "Digi-Key PN"
 	1    1600 3070
 	-1   0    0    -1
@@
 F 2 "Custom Footprints Library:Keystone_8191" H 1600 3420 50  0001 C CNN
 F 3 "~" H 1600 3420 50  0001 C CNN
+F 4 "36-8191-ND" H 0   0   50  0001 C CNN "Digi-Key PN"
 	1    1600 3420
 	-1   0    0    -1
@@
 F 2 "Custom Footprints Library:Keystone_8191" H 1600 4070 50  0001 C CNN
 F 3 "~" H 1600 4070 50  0001 C CNN
+F 4 "36-8191-ND" H 0   0   50  0001 C CNN "Digi-Key PN"
 	1    1600 4070
 	-1   0    0    -1
@@
 F 2 "Custom Footprints Library:Keystone_8191" H 1600 3720 50  0001 C CNN
 F 3 "~" H 1600 3720 50  0001 C CNN
+F 4 "36-8191-ND" H 0   0   50  0001 C CNN "Digi-Key PN"
 	1    1600 3720
 	-1   0    0    -1
@@
 F 2 "Fuse_Holders_and_Fuses:Fuse_SMD1206_Reflow" V 2250 2450 50  0001 C CNN
 F 3 "~" H 2320 2450 50  0001 C CNN
+F 4 "507-1946-1-ND" H 0   0   50  0001 C CNN "Digi-Key PN"
 	1    2320 2450
 	0    1    1    0
@@
 F 3 "" H 7025 4420 50  0001 C CNN
 F 4 "0603" H 6850 4420 50  0001 R CNN "display_footprint"
-F 5 "25V" H 6850 4320 50  0001 R CNN "Voltage"
+F 5 "50V" H 6850 4320 50  0001 R CNN "Voltage"
 F 6 "X7R" H 6850 4220 50  0001 R CNN "Dielectric"
-F 7 "PN" H 7425 4820 60  0001 C CNN "Digi-Key PN"
+F 7 "1276-1921-1-ND" H 7425 4820 60  0001 C CNN "Digi-Key PN"
 	1    7000 4320
 	1    0    0    -1
@@
 F 5 "1%" H 9130 4840 50  0000 L CNN "Tolerance"
 F 6 "1/10W" H 9130 4760 50  0000 L CNN "Wattage"
-F 7 "PN" H 9350 5240 60  0001 C CNN "Digi-Key PN"
+F 7 "RHM1.0KDCT-ND" H 9350 5240 60  0001 C CNN "Digi-Key PN"
 	1    9050 4840
 	-1   0    0    -1
@@
 F 2 "" H 9050 4540 50  0001 C CNN
 F 3 "~" H 9050 4540 50  0001 C CNN
+F 4 "160-1446-1-ND" H 0   0   50  0001 C CNN "Digi-Key PN"
 	1    9050 4540
 	0    -1   -1   0
@@
 F 5 "50V" H 7790 5540 50  0000 R CNN "Voltage"
 F 6 "X7R" H 7790 5440 50  0000 R CNN "Dielectric"
-F 7 "PN" H 8365 6040 60  0001 C CNN "Digi-Key PN"
+F 7 "490-4779-1-ND" H 8365 6040 60  0001 C CNN "Digi-Key PN"
 	1    7940 5540
 	1    0    0    -1

Commit message: Assigned footprints
Parts:
- C201, C202, C203, C205, C207: footprint (none) -> Capacitors_SMD:C_0603
- C204, C206, C208: footprint (none) -> Capacitors_Tantalum_SMD:CP_Tantalum_Case-X_EIA-7343-43_Reflow
- D202: footprint (none) -> LEDs:LED_0603
- Q201, Q202: footprint Package_TO_SOT_SMD:TDSON-8-1 -> TO_SOT_Packages_SMD:TDSON-8-1
- R201, R202, R203, R204, R205, R206, R207, R208, R209: footprint (none) -> Resistors_SMD:R_0603
- TP201: footprint (none) -> Pin_Headers:Pin_Header_Angled_1x01_Pitch2.54mm
- TP202: footprint (none) -> Measurement_Points:Measurement_Point_Round-SMD-Pad_Small
- U201: footprint Package_DFN_QFN:DFN-8-1EP_2x3mm_P0.5mm_EP0.61x2.2mm -> Housings_DFN_QFN:DFN-8-1EP_2x3mm_Pitch0.5mm
Changed lines of the file:
@@
 F 0 "R201" H 2740 4530 50  0000 R CNN
 F 1 "6.04M" V 2840 4530 50  0000 C CNN
-F 2 "" H 2840 4530 50  0001 C CNN
+F 2 "Resistors_SMD:R_0603" H 2840 4530 50  0001 C CNN
 F 3 "" H 2840 4530 50  0001 C CNN
 F 4 "0603" H 2920 4610 50  0000 L CNN "display_footprint"
@@
 F 0 "C201" H 5175 6370 50  0000 L CNN
 F 1 "0.1uF" H 5175 6170 50  0000 L CNN
-F 2 "" H 5188 6120 50  0001 C CNN
+F 2 "Capacitors_SMD:C_0603" H 5188 6120 50  0001 C CNN
 F 3 "" H 5175 6370 50  0001 C CNN
 F 4 "0603" H 5000 6370 50  0000 R CNN "display_footprint"
@@
 F 0 "C202" H 5475 6370 50  0000 L CNN
 F 1 "10nF" H 5475 6170 50  0000 L CNN
-F 2 "" H 5488 6120 50  0001 C CNN
+F 2 "Capacitors_SMD:C_0603" H 5488 6120 50  0001 C CNN
 F 3 "" H 5475 6370 50  0001 C CNN
 F 4 "0603" H 5300 6370 50  0001 R CNN "display_footprint"
@@
 F 0 "C203" H 5775 6370 50  0000 L CNN
 F 1 "1nF" H 5775 6170 50  0000 L CNN
-F 2 "" H 5788 6120 50  0001 C CNN
+F 2 "Capacitors_SMD:C_0603" H 5788 6120 50  0001 C CNN
 F 3 "" H 5775 6370 50  0001 C CNN
 F 4 "0603" H 5600 6370 50  0001 R CNN "display_footprint"
@@
 F 0 "R202" H 2740 5060 50  0000 R CNN
 F 1 "86.6k" V 2840 5060 40  0000 C CNN
-F 2 "" H 2840 5060 50  0001 C CNN
+F 2 "Resistors_SMD:R_0603" H 2840 5060 50  0001 C CNN
 F 3 "" H 2840 5060 50  0001 C CNN
 F 4 "0603" H 2920 5140 50  0000 L CNN "display_footprint"
@@
 F 0 "R203" H 2740 5560 50  0000 R CNN
 F 1 "243k" V 2840 5560 40  0000 C CNN
-F 2 "" H 2840 5560 50  0001 C CNN
+F 2 "Resistors_SMD:R_0603" H 2840 5560 50  0001 C CNN
 F 3 "" H 2840 5560 50  0001 C CNN
 F 4 "0603" H 2920 5640 50  0000 L CNN "display_footprint"
@@
 F 0 "R204" H 3270 4040 50  0000 R CNN
 F 1 "100k" V 3370 4040 40  0000 C CNN
-F 2 "" H 3370 4040 50  0001 C CNN
+F 2 "Resistors_SMD:R_0603" H 3370 4040 50  0001 C CNN
 F 3 "" H 3370 4040 50  0001 C CNN
 F 4 "0603" H 3450 4120 50  0000 L CNN "display_footprint"
@@
 F 0 "R205" V 4820 3110 50  0000 C CNN
 F 1 "10" V 4920 3110 50  0000 C CNN
-F 2 "" H 4920 3110 50  0001 C CNN
+F 2 "Resistors_SMD:R_0603" H 4920 3110 50  0001 C CNN
 F 3 "" H 4920 3110 50  0001 C CNN
 F 4 "0603" V 5020 3110 50  0000 C CNN "display_footprint"
@@
 F 0 "R206" V 5690 3110 50  0000 C CNN
 F 1 "10" V 5790 3110 50  0000 C CNN
-F 2 "" H 5790 3110 50  0001 C CNN
+F 2 "Resistors_SMD:R_0603" H 5790 3110 50  0001 C CNN
 F 3 "" H 5790 3110 50  0001 C CNN
 F 4 "0603" V 5890 3110 50  0000 C CNN "display_footprint"
@@
 F 0 "R208" H 6900 4020 50  0000 R CNN
 F 1 "5.1k" V 7000 4020 50  0000 C CNN
-F 2 "" H 7000 4020 50  0001 C CNN
+F 2 "Resistors_SMD:R_0603" H 7000 4020 50  0001 C CNN
 F 3 "" H 7000 4020 50  0001 C CNN
 F 4 "0603" H 7080 4100 50  0000 L CNN "display_footprint"
@@
 F 0 "U201" H 5060 5440 50  0000 L CNN
 F 1 "LTC4365DDB" H 5410 5440 50  0000 L CNN
-F 2 "Package_DFN_QFN:DFN-8-1EP_2x3mm_P0.5mm_EP0.61x2.2mm" H 5360 4540 50  0001 C CNN
+F 2 "Housings_DFN_QFN:DFN-8-1EP_2x3mm_Pitch0.5mm" H 5360 4540 50  0001 C CNN
 F 3 "http://cds.linear.com/docs/en/datasheet/4365fa.pdf" H 5360 4790 50  0001 C CNN
 F 4 "LTC4365IDDB#TRMPBFCT-ND" H 5360 4540 50  0001 C CNN "Digi-Key PN"
@@
 F 0 "C204" H 7025 3050 50  0000 L CNN
 F 1 "100uF" H 7025 2850 50  0000 L CNN
-F 2 "" H 7038 2800 50  0001 C CNN
+F 2 "Capacitors_Tantalum_SMD:CP_Tantalum_Case-X_EIA-7343-43_Reflow" H 7038 2800 50  0001 C CNN
 F 3 "" H 7025 3050 50  0001 C CNN
 F 4 "718-1102-1-ND" H 7000 2950 50  0001 C CNN "Digi-Key PN"
@@
 F 0 "C206" H 7775 3050 50  0000 L CNN
 F 1 "100uF" H 7775 2850 50  0000 L CNN
-F 2 "" H 7788 2800 50  0001 C CNN
+F 2 "Capacitors_Tantalum_SMD:CP_Tantalum_Case-X_EIA-7343-43_Reflow" H 7788 2800 50  0001 C CNN
 F 3 "" H 7775 3050 50  0001 C CNN
 F 4 "718-1102-1-ND" H 7750 2950 50  0001 C CNN "Digi-Key PN"
@@
 F 0 "C208" H 8525 3050 50  0000 L CNN
 F 1 "100uF" H 8525 2850 50  0000 L CNN
-F 2 "" H 8538 2800 50  0001 C CNN
+F 2 "Capacitors_Tantalum_SMD:CP_Tantalum_Case-X_EIA-7343-43_Reflow" H 8538 2800 50  0001 C CNN
 F 3 "" H 8525 3050 50  0001 C CNN
 F 4 "718-1102-1-ND" H 8500 2950 50  0001 C CNN "Digi-Key PN"
@@
 F 0 "R207" H 5950 4410 50  0000 R CNN
 F 1 "10k" V 6050 4410 50  0000 C CNN
-F 2 "" H 6050 4410 50  0001 C CNN
+F 2 "Resistors_SMD:R_0603" H 6050 4410 50  0001 C CNN
 F 3 "" H 6050 4410 50  0001 C CNN
 F 4 "0603" H 6130 4490 50  0000 L CNN "display_footprint"
@@
 F 0 "TP202" H 7000 2800 50  0000 C CNN
 F 1 "TP" H 7000 2800 50  0001 C CNN
-F 2 "" H 7000 2650 60  0000 C CNN
+F 2 "Measurement_Points:Measurement_Point_Round-SMD-Pad_Small" H 7000 2650 60  0001 C CNN
 F 3 "" H 7000 2650 60  0000 C CNN
 	1    7000 2650
@@
 F 0 "TP201" H 1880 5200 50  0000 C CNN
 F 1 "TP" H 1880 5200 50  0001 C CNN
-F 2 "" H 1880 5050 60  0000 C CNN
+F 2 "Pin_Headers:Pin_Header_Angled_1x01_Pitch2.54mm" H 1880 5050 60  0001 C CNN
 F 3 "" H 1880 5050 60  0000 C CNN
 	1    1880 5050
@@
 F 0 "Q201" V 5033 2820 50  0000 C CNN
 F 1 "BSC123N10LSGATMA1" V 4942 2820 50  0000 C CNN
-F 2 "Package_TO_SOT_SMD:TDSON-8-1" H 4890 2745 50  0001 L CIN
+F 2 "TO_SOT_Packages_SMD:TDSON-8-1" H 4890 2745 50  0001 L CIN
 F 3 "http://www.infineon.com/dgdl/Infineon-BSC123N10LS-DS-v02_08-en.pdf?fileId=db3a30431b3e89eb011b4626974b7df5" V 4690 2820 50  0001 L CNN
 F 4 "BSC123N10LSGATMA1CT-ND" H 4690 2820 50  0001 C CNN "Digi-Key PN"
@@
 F 0 "Q202" V 6383 2820 50  0000 C CNN
 F 1 "BSC123N10LSGATMA1" V 6292 2820 50  0000 C CNN
-F 2 "Package_TO_SOT_SMD:TDSON-8-1" H 6240 2745 50  0001 L CIN
+F 2 "TO_SOT_Packages_SMD:TDSON-8-1" H 6240 2745 50  0001 L CIN
 F 3 "http://www.infineon.com/dgdl/Infineon-BSC123N10LS-DS-v02_08-en.pdf?fileId=db3a30431b3e89eb011b4626974b7df5" V 6040 2820 50  0001 L CNN
 F 4 "BSC123N10LSGATMA1CT-ND" H 6040 2820 50  0001 C CNN "Digi-Key PN"
@@
 F 0 "C205" H 7025 4420 50  0000 L CNN
 F 1 "10nF" H 7025 4220 50  0000 L CNN
-F 2 "" H 7038 4170 50  0001 C CNN
+F 2 "Capacitors_SMD:C_0603" H 7038 4170 50  0001 C CNN
 F 3 "" H 7025 4420 50  0001 C CNN
 F 4 "0603" H 6850 4420 50  0001 R CNN "display_footprint"
@@
 F 0 "R209" H 8950 4840 50  0000 R CNN
 F 1 "1k" V 9050 4840 50  0000 C CNN
-F 2 "" H 9050 4840 50  0001 C CNN
+F 2 "Resistors_SMD:R_0603" H 9050 4840 50  0001 C CNN
 F 3 "" H 9050 4840 50  0001 C CNN
 F 4 "0603" H 9130 4920 50  0000 L CNN "display_footprint"
@@
 F 0 "D202" H 9050 4640 50  0000 C CNN
 F 1 "Green" H 9050 4440 50  0000 C CNN
-F 2 "" H 9050 4540 50  0001 C CNN
+F 2 "LEDs:LED_0603" H 9050 4540 50  0001 C CNN
 F 3 "~" H 9050 4540 50  0001 C CNN
 F 4 "160-1446-1-ND" H 0   0   50  0001 C CNN "Digi-Key PN"
@@
 F 0 "C207" H 7965 5640 50  0000 L CNN
 F 1 "0.1uF" H 7965 5440 50  0000 L CNN
-F 2 "" H 7978 5390 50  0001 C CNN
+F 2 "Capacitors_SMD:C_0603" H 7978 5390 50  0001 C CNN
 F 3 "" H 7965 5640 50  0001 C CNN
 F 4 "0603" H 7790 5640 50  0000 R CNN "display_footprint"
