File: hdw/LTC7851_Demo/Power_Input.sch (KiCad schematic (older format))
At the start: 33 parts, among them J201 +12VIN, J202 +12VIN, J203 +12VIN, J204 GNDIN, J205 GNDIN, J206 GNDIN, Q201 BSC123N10LSGATMA1, Q202 BSC123N10LSGATMA1, U201 LTC4365DDB, U202 74LVC1G06

Commit message: Added page titles
Other:
- note added: "Power Input"
Changed lines of the file:
@@
 Text GLabel 8040 5140 0    50   Input ~ 0
 POS12_PGOOD
+Text Notes 540  690  0    100  ~ 20
+Power Input
 $EndSCHEMATC

Commit message: Finished arranging parts on board
Parts:
- removed J202, J203: +12VIN, Custom Footprints Library:Keystone_8191, symbol Connector:Screw_Terminal_01x01
- removed J204, J205: GNDIN, Custom Footprints Library:Keystone_8191, symbol Connector:Screw_Terminal_01x01
- J201: value +12VIN -> +12V IN; footprint Custom Footprints Library:Keystone_8191 -> Custom Footprints Library:Wuerth_7461096_M4_Shank_9pos; Digi-Key PN 36-8191-ND -> 732-3214-ND
- J206: value GNDIN -> GND IN; footprint Custom Footprints Library:Keystone_8191 -> Custom Footprints Library:Wuerth_7461096_M4_Shank_9pos; Digi-Key PN 36-8191-ND -> 732-3214-ND
Connections:
- wire segments 83 -> 74
Changed lines of the file:
@@
 AR Path="/5BB86F23/5BB576E9" Ref="R201"  Part="1"
 F 0 "R201" H 2740 4530 50  0000 R CNN
-F 1 "6.04M" V 2840 4530 50  0000 C CNN
+F 1 "6.04M" V 2840 4530 40  0000 C CNN
 F 2 "Resistors_SMD:R_0603" H 2840 4530 50  0001 C CNN
 F 3 "" H 2840 4530 50  0001 C CNN
@@
 $EndComp
 $Comp
-L Connector:Screw_Terminal_01x01 J201
-U 1 1 5BB6951A
-P 1600 2720
-F 0 "J201" H 1600 2820 50  0000 C CNN
-F 1 "+12VIN" H 1600 2620 50  0000 C CNN
-F 2 "Custom Footprints Library:Keystone_8191" H 1600 2720 50  0001 C CNN
-F 3 "~" H 1600 2720 50  0001 C CNN
-F 4 "36-8191-ND" H 0   0   50  0001 C CNN "Digi-Key PN"
-	1    1600 2720
-	-1   0    0    -1
-$EndComp
-Wire Wire Line
-	1800 2720 1880 2720
-$Comp
-L Connector:Screw_Terminal_01x01 J206
-U 1 1 5BB69E61
-P 1600 4420
-F 0 "J206" H 1600 4520 50  0000 C CNN
-F 1 "GNDIN" H 1600 4320 50  0000 C CNN
-F 2 "Custom Footprints Library:Keystone_8191" H 1600 4420 50  0001 C CNN
-F 3 "~" H 1600 4420 50  0001 C CNN
-F 4 "36-8191-ND" H 0   0   50  0001 C CNN "Digi-Key PN"
-	1    1600 4420
-	-1   0    0    -1
-$EndComp
-$Comp
 L power:GND #PWR0201
 U 1 1 5BB6A1CD
-P 1880 4500
-F 0 "#PWR0201" H 1880 4250 50  0001 C CNN
-F 1 "GND" H 1880 4350 50  0000 C CNN
-F 2 "" H 1880 4500 50  0001 C CNN
-F 3 "" H 1880 4500 50  0001 C CNN
-	1    1880 4500
-	1    0    0    -1
-$EndComp
-Wire Wire Line
-	1880 4500 1880 4420
-Wire Wire Line
-	1880 4420 1800 4420
+P 1880 3330
+F 0 "#PWR0201" H 1880 3080 50  0001 C CNN
+F 1 "GND" H 1880 3180 50  0000 C CNN
+F 2 "" H 1880 3330 50  0001 C CNN
+F 3 "" H 1880 3330 50  0001 C CNN
+	1    1880 3330
+	1    0    0    -1
+$EndComp
+Wire Wire Line
+	1880 3330 1880 3250
+Wire Wire Line
+	1880 3250 1800 3250
 Wire Wire Line
 	5760 3790 6560 3790
@@
 L power:GND #PWR0203
 U 1 1 5BB7FEE9
-P 2100 4500
-F 0 "#PWR0203" H 2100 4250 50  0001 C CNN
-F 1 "GND" H 2100 4350 50  0000 C CNN
-F 2 "" H 2100 4500 50  0001 C CNN
-F 3 "" H 2100 4500 50  0001 C CNN
-	1    2100 4500
+P 2100 3330
+F 0 "#PWR0203" H 2100 3080 50  0001 C CNN
+F 1 "GND" H 2100 3180 50  0000 C CNN
+F 2 "" H 2100 3330 50  0001 C CNN
+F 3 "" H 2100 3330 50  0001 C CNN
+	1    2100 3330
 	1    0    0    -1
 $EndComp
@@
 L power:PWR_FLAG #FLG0201
 U 1 1 5BB80368
-P 2100 4500
-F 0 "#FLG0201" H 2100 4575 50  0001 C CNN
-F 1 "PWR_FLAG" H 2100 4650 50  0000 C CNN
-F 2 "" H 2100 4500 50  0001 C CNN
-F 3 "~" H 2100 4500 50  0001 C CNN
-	1    2100 4500
+P 2100 3330
+F 0 "#FLG0201" H 2100 3405 50  0001 C CNN
+F 1 "PWR_FLAG" H 2100 3480 50  0000 C CNN
+F 2 "" H 2100 3330 50  0001 C CNN
+F 3 "~" H 2100 3330 50  0001 C CNN
+	1    2100 3330
 	1    0    0    -1
 $EndComp
@@
 L Custom_Library:TP TP201
 U 1 1 5BB80406
-P 1880 5050
-F 0 "TP201" H 1880 5200 50  0000 C CNN
-F 1 "TP" H 1880 5200 50  0001 C CNN
-F 2 "Pin_Headers:Pin_Header_Angled_1x01_Pitch2.54mm" H 1880 5050 60  0001 C CNN
-F 3 "" H 1880 5050 60  0000 C CNN
-	1    1880 5050
+P 1880 3880
+F 0 "TP201" H 1880 4030 50  0000 C CNN
+F 1 "TP" H 1880 4030 50  0001 C CNN
+F 2 "Pin_Headers:Pin_Header_Angled_1x01_Pitch2.54mm" H 1880 3880 60  0001 C CNN
+F 3 "" H 1880 3880 60  0000 C CNN
+	1    1880 3880
 	1    0    0    -1
 $EndComp
@@
 L power:GND #PWR0202
 U 1 1 5BB80478
-P 1880 5050
-F 0 "#PWR0202" H 1880 4800 50  0001 C CNN
-F 1 "GND" H 1880 4900 50  0000 C CNN
-F 2 "" H 1880 5050 50  0001 C CNN
-F 3 "" H 1880 5050 50  0001 C CNN
-	1    1880 5050
+P 1880 3880
+F 0 "#PWR0202" H 1880 3630 50  0001 C CNN
+F 1 "GND" H 1880 3730 50  0000 C CNN
+F 2 "" H 1880 3880 50  0001 C CNN
+F 3 "" H 1880 3880 50  0001 C CNN
+	1    1880 3880
 	1    0    0    -1
 $EndComp
@@
 Wire Wire Line
 	2840 2640 2840 2720
-$Comp
-L Connector:Screw_Terminal_01x01 J202
-U 1 1 5BB97294
-P 1600 3070
-F 0 "J202" H 1600 3170 50  0000 C CNN
-F 1 "+12VIN" H 1600 2970 50  0000 C CNN
-F 2 "Custom Footprints Library:Keystone_8191" H 1600 3070 50  0001 C CNN
-F 3 "~" H 1600 3070 50  0001 C CNN
-F 4 "36-8191-ND" H 0   0   50  0001 C CNN "Digi-Key PN"
-	1    1600 3070
-	-1   0    0    -1
-$EndComp
-$Comp
-L Connector:Screw_Terminal_01x01 J203
-U 1 1 5BB972F4
-P 1600 3420
-F 0 "J203" H 1600 3520 50  0000 C CNN
-F 1 "+12VIN" H 1600 3320 50  0000 C CNN
-F 2 "Custom Footprints Library:Keystone_8191" H 1600 3420 50  0001 C CNN
-F 3 "~" H 1600 3420 50  0001 C CNN
-F 4 "36-8191-ND" H 0   0   50  0001 C CNN "Digi-Key PN"
-	1    1600 3420
-	-1   0    0    -1
-$EndComp
-Wire Wire Line
-	1800 3420 1880 3420
-Wire Wire Line
-	1880 3420 1880 3070
-Connection ~ 1880 2720
-Wire Wire Line
-	1880 2720 2130 2720
-Wire Wire Line
-	1800 3070 1880 3070
-Connection ~ 1880 3070
-Wire Wire Line
-	1880 3070 1880 2720
-$Comp
-L Connector:Screw_Terminal_01x01 J205
-U 1 1 5BB99C26
-P 1600 4070
-F 0 "J205" H 1600 4170 50  0000 C CNN
-F 1 "GNDIN" H 1600 3970 50  0000 C CNN
-F 2 "Custom Footprints Library:Keystone_8191" H 1600 4070 50  0001 C CNN
-F 3 "~" H 1600 4070 50  0001 C CNN
-F 4 "36-8191-ND" H 0   0   50  0001 C CNN "Digi-Key PN"
-	1    1600 4070
-	-1   0    0    -1
-$EndComp
-$Comp
-L Connector:Screw_Terminal_01x01 J204
-U 1 1 5BB99C80
-P 1600 3720
-F 0 "J204" H 1600 3820 50  0000 C CNN
-F 1 "GNDIN" H 1600 3620 50  0000 C CNN
-F 2 "Custom Footprints Library:Keystone_8191" H 1600 3720 50  0001 C CNN
-F 3 "~" H 1600 3720 50  0001 C CNN
-F 4 "36-8191-ND" H 0   0   50  0001 C CNN "Digi-Key PN"
-	1    1600 3720
-	-1   0    0    -1
-$EndComp
-Wire Wire Line
-	1800 3720 1880 3720
-Wire Wire Line
-	1880 3720 1880 4070
-Connection ~ 1880 4420
-Wire Wire Line
-	1800 4070 1880 4070
-Connection ~ 1880 4070
-Wire Wire Line
-	1880 4070 1880 4420
 $Comp
 L Custom_Library:+5.5V_MNG #PWR0210
@@
 Text Notes 540  690  0    100  ~ 20
 Power Input
+Wire Wire Line
+	1800 2720 2130 2720
+$Comp
+L Connector:Screw_Terminal_01x01 J?
+U 1 1 5BC409E0
+P 1600 2720
+AR Path="/5BB9D026/5BC409E0" Ref="J?"  Part="1"
+AR Path="/5BB86F23/5BC409E0" Ref="J201"  Part="1"
+F 0 "J201" H 1600 2820 50  0000 C CNN
+F 1 "+12V IN" H 1600 2620 50  0000 C CNN
+F 2 "Custom Footprints Library:Wuerth_7461096_M4_Shank_9pos" H 1600 2720 50  0001 C CNN
+F 3 "~" H 1600 2720 50  0001 C CNN
+F 4 "732-3214-ND" H -3920 70  50  0001 C CNN "Digi-Key PN"
+	1    1600 2720
+	-1   0    0    -1
+$EndComp
+$Comp
+L Connector:Screw_Terminal_01x01 J?
+U 1 1 5BC43E0D
+P 1600 3250
+AR Path="/5BB9D026/5BC43E0D" Ref="J?"  Part="1"
+AR Path="/5BB86F23/5BC43E0D" Ref="J206"  Part="1"
+F 0 "J206" H 1600 3350 50  0000 C CNN
+F 1 "GND IN" H 1600 3150 50  0000 C CNN
+F 2 "Custom Footprints Library:Wuerth_7461096_M4_Shank_9pos" H 1600 3250 50  0001 C CNN
+F 3 "~" H 1600 3250 50  0001 C CNN
+F 4 "732-3214-ND" H -3920 600 50  0001 C CNN "Digi-Key PN"
+	1    1600 3250
+	-1   0    0    -1
+$EndComp
 $EndSCHEMATC

Commit message: Added a few connectors and cleaned up some routing
Parts:
- removed F201, F202: 25A, Fuse_Holders_and_Fuses:Fuse_SMD1206_Reflow, symbol Device:Fuse
- Q201, Q202: value BSC123N10LSGATMA1 -> IPC100N04S51R7ATMA1
Connections:
- wire segments 74 -> 67
Changed lines of the file:
@@
 Wire Wire Line
 	4410 2720 4490 2720
-$Comp
-L Device:Fuse F202
-U 1 1 5BB64ED2
-P 2320 2720
-F 0 "F202" V 2400 2720 50  0000 C CNN
-F 1 "25A" V 2245 2720 50  0000 C CNN
-F 2 "Fuse_Holders_and_Fuses:Fuse_SMD1206_Reflow" V 2250 2720 50  0001 C CNN
-F 3 "~" H 2320 2720 50  0001 C CNN
-F 4 "507-1946-1-ND" H 0   0   50  0001 C CNN "Digi-Key PN"
-	1    2320 2720
-	0    1    1    0
-$EndComp
-Wire Wire Line
-	2470 2720 2510 2720
 Connection ~ 2840 2720
 $Comp
@@
 $EndComp
 $Comp
-L Device:Fuse F201
-U 1 1 5BC39D4F
-P 2320 2450
-F 0 "F201" V 2400 2450 50  0000 C CNN
-F 1 "25A" V 2245 2450 50  0000 C CNN
-F 2 "Fuse_Holders_and_Fuses:Fuse_SMD1206_Reflow" V 2250 2450 50  0001 C CNN
-F 3 "~" H 2320 2450 50  0001 C CNN
-F 4 "507-1946-1-ND" H 0   0   50  0001 C CNN "Digi-Key PN"
-	1    2320 2450
-	0    1    1    0
-$EndComp
-Wire Wire Line
-	2170 2450 2130 2450
-Wire Wire Line
-	2130 2450 2130 2720
-Connection ~ 2130 2720
-Wire Wire Line
-	2130 2720 2170 2720
-Wire Wire Line
-	2470 2450 2510 2450
-Wire Wire Line
-	2510 2450 2510 2720
-Connection ~ 2510 2720
-Wire Wire Line
-	2510 2720 2840 2720
-$Comp
 L Transistor_FET:BSC123N10LSG Q?
 U 1 1 5BC3F351
@@
 AR Path="/5BB86F23/5BC3F351" Ref="Q201"  Part="1"
 F 0 "Q201" V 5033 2820 50  0000 C CNN
-F 1 "BSC123N10LSGATMA1" V 4942 2820 50  0000 C CNN
+F 1 "IPC100N04S51R7ATMA1" V 4942 2820 50  0000 C CNN
 F 2 "TO_SOT_Packages_SMD:TDSON-8-1" H 4890 2745 50  0001 L CIN
 F 3 "http://www.infineon.com/dgdl/Infineon-BSC123N10LS-DS-v02_08-en.pdf?fileId=db3a30431b3e89eb011b4626974b7df5" V 4690 2820 50  0001 L CNN
@@
 AR Path="/5BB86F23/5BC46F59" Ref="Q202"  Part="1"
 F 0 "Q202" V 6383 2820 50  0000 C CNN
-F 1 "BSC123N10LSGATMA1" V 6292 2820 50  0000 C CNN
+F 1 "IPC100N04S51R7ATMA1" V 6292 2820 50  0000 C CNN
 F 2 "TO_SOT_Packages_SMD:TDSON-8-1" H 6240 2745 50  0001 L CIN
 F 3 "http://www.infineon.com/dgdl/Infineon-BSC123N10LS-DS-v02_08-en.pdf?fileId=db3a30431b3e89eb011b4626974b7df5" V 6040 2820 50  0001 L CNN
@@
 Text Notes 540  690  0    100  ~ 20
 Power Input
-Wire Wire Line
-	1800 2720 2130 2720
 $Comp
 L Connector:Screw_Terminal_01x01 J?
@@
 	-1   0    0    -1
 $EndComp
+Wire Wire Line
+	2840 2720 1800 2720
 $EndSCHEMATC
