File: hdw/LTC7851_Demo/Mechanical.sch (KiCad schematic (older format))
At the start: 24 parts

Commit message: Duplicated master phase, added status LEDs and a few test points
Parts:
- removed MH? (x8): MountingHole, Mounting_Holes:MountingHole_3mm_Pad_Via, symbol Mechanical:MountingHole_Pad
- removed MK? (x2): 4-40 Screw, symbol Custom_Library:Screw
- removed MK? (x2): 4-40 Standoff, symbol Custom_Library:Standoff
- added MH? (x6): MountingHole, symbol Mechanical:MountingHole
Connections:
- net labels removed: Earth_Protective

Commit message: Filled in power input page
Changed lines of the file:
@@
 Mounting Holes and Mechanical Components
-$Comp
-L Custom_Library:MU_Logo #G?
-U 1 1 5BB6A5D4
-P 9900 1100
-F 0 "#G?" H 9900 614 60  0001 C CNN
-F 1 "MU_Logo" H 9900 1586 60  0001 C CNN
-F 2 "" H 9900 1100 50  0001 C CNN
-F 3 "" H 9900 1100 50  0001 C CNN
-	1    9900 1100
-	1    0    0    -1
-$EndComp
 $Comp
 L Custom_Library:Screw MK?

Commit message: Annotated schematic
Parts:
- gave numbers to parts that had none: 18
Changed lines of the file:
@@
 Mounting Holes and Mechanical Components
 $Comp
-L Custom_Library:Screw MK?
+L Custom_Library:Screw MK1001
 U 1 1 5BC10ED5
 P 6470 2210
-F 0 "MK?" H 6470 2310 50  0000 C CNN
+F 0 "MK1001" H 6470 2310 50  0000 C CNN
 F 1 "4-40 Screw" H 6470 2410 50  0000 C CNN
 F 2 "" H 6470 2460 50  0001 C CNN
@@
 $EndComp
 $Comp
-L Custom_Library:Screw MK?
+L Custom_Library:Screw MK1005
 U 1 1 5BC1118A
 P 7220 2210
-F 0 "MK?" H 7220 2310 50  0000 C CNN
+F 0 "MK1005" H 7220 2310 50  0000 C CNN
 F 1 "4-40 Screw" H 7220 2410 50  0000 C CNN
 F 2 "" H 7220 2460 50  0001 C CNN
@@
 $EndComp
 $Comp
-L Custom_Library:Screw MK?
+L Custom_Library:Screw MK1009
 U 1 1 5BC11270
 P 7970 2210
-F 0 "MK?" H 7970 2310 50  0000 C CNN
+F 0 "MK1009" H 7970 2310 50  0000 C CNN
 F 1 "4-40 Screw" H 7970 2410 50  0000 C CNN
 F 2 "" H 7970 2460 50  0001 C CNN
@@
 $EndComp
 $Comp
-L Custom_Library:Screw MK?
+L Custom_Library:Screw MK1002
 U 1 1 5BC113EE
 P 6470 2960
-F 0 "MK?" H 6470 3060 50  0000 C CNN
+F 0 "MK1002" H 6470 3060 50  0000 C CNN
 F 1 "4-40 Screw" H 6470 3160 50  0000 C CNN
 F 2 "" H 6470 3210 50  0001 C CNN
@@
 $EndComp
 $Comp
-L Custom_Library:Screw MK?
+L Custom_Library:Screw MK1006
 U 1 1 5BC113F5
 P 7220 2960
-F 0 "MK?" H 7220 3060 50  0000 C CNN
+F 0 "MK1006" H 7220 3060 50  0000 C CNN
 F 1 "4-40 Screw" H 7220 3160 50  0000 C CNN
 F 2 "" H 7220 3210 50  0001 C CNN
@@
 $EndComp
 $Comp
-L Custom_Library:Screw MK?
+L Custom_Library:Screw MK1010
 U 1 1 5BC113FC
 P 7970 2960
-F 0 "MK?" H 7970 3060 50  0000 C CNN
+F 0 "MK1010" H 7970 3060 50  0000 C CNN
 F 1 "4-40 Screw" H 7970 3160 50  0000 C CNN
 F 2 "" H 7970 3210 50  0001 C CNN
@@
 $EndComp
 $Comp
-L Custom_Library:Standoff MK?
+L Custom_Library:Standoff MK1003
 U 1 1 5BC1193F
 P 6470 3720
-F 0 "MK?" H 6470 3870 50  0000 C CNN
+F 0 "MK1003" H 6470 3870 50  0000 C CNN
 F 1 "4-40 Standoff" H 6470 3970 50  0000 C CNN
 F 2 "" H 6470 4070 50  0001 C CNN
@@
 $EndComp
 $Comp
-L Custom_Library:Standoff MK?
+L Custom_Library:Standoff MK1007
 U 1 1 5BC12310
 P 7220 3720
-F 0 "MK?" H 7220 3870 50  0000 C CNN
+F 0 "MK1007" H 7220 3870 50  0000 C CNN
 F 1 "4-40 Standoff" H 7220 3970 50  0000 C CNN
 F 2 "" H 7220 4070 50  0001 C CNN
@@
 $EndComp
 $Comp
-L Custom_Library:Standoff MK?
+L Custom_Library:Standoff MK1011
 U 1 1 5BC1235A
 P 7970 3720
-F 0 "MK?" H 7970 3870 50  0000 C CNN
+F 0 "MK1011" H 7970 3870 50  0000 C CNN
 F 1 "4-40 Standoff" H 7970 3970 50  0000 C CNN
 F 2 "" H 7970 4070 50  0001 C CNN
@@
 $EndComp
 $Comp
-L Custom_Library:Standoff MK?
+L Custom_Library:Standoff MK1004
 U 1 1 5BC12534
 P 6470 4470
-F 0 "MK?" H 6470 4620 50  0000 C CNN
+F 0 "MK1004" H 6470 4620 50  0000 C CNN
 F 1 "4-40 Standoff" H 6470 4720 50  0000 C CNN
 F 2 "" H 6470 4820 50  0001 C CNN
@@
 $EndComp
 $Comp
-L Custom_Library:Standoff MK?
+L Custom_Library:Standoff MK1008
 U 1 1 5BC1253B
 P 7220 4470
-F 0 "MK?" H 7220 4620 50  0000 C CNN
+F 0 "MK1008" H 7220 4620 50  0000 C CNN
 F 1 "4-40 Standoff" H 7220 4720 50  0000 C CNN
 F 2 "" H 7220 4820 50  0001 C CNN
@@
 $EndComp
 $Comp
-L Custom_Library:Standoff MK?
+L Custom_Library:Standoff MK1012
 U 1 1 5BC12542
 P 7970 4470
-F 0 "MK?" H 7970 4620 50  0000 C CNN
+F 0 "MK1012" H 7970 4620 50  0000 C CNN
 F 1 "4-40 Standoff" H 7970 4720 50  0000 C CNN
 F 2 "" H 7970 4820 50  0001 C CNN
@@
 $EndComp
 $Comp
-L Mechanical:MountingHole MH?
+L Mechanical:MountingHole MH1001
 U 1 1 5BD5283B
 P 1830 2260
-F 0 "MH?" H 1830 2460 50  0000 C CNN
+F 0 "MH1001" H 1830 2460 50  0000 C CNN
 F 1 "MountingHole" H 1830 2385 50  0000 C CNN
 F 2 "" H 1830 2260 50  0001 C CNN
@@
 $EndComp
 $Comp
-L Mechanical:MountingHole MH?
+L Mechanical:MountingHole MH1003
 U 1 1 5BD52910
 P 2580 2260
-F 0 "MH?" H 2580 2460 50  0000 C CNN
+F 0 "MH1003" H 2580 2460 50  0000 C CNN
 F 1 "MountingHole" H 2580 2385 50  0000 C CNN
 F 2 "" H 2580 2260 50  0001 C CNN
@@
 $EndComp
 $Comp
-L Mechanical:MountingHole MH?
+L Mechanical:MountingHole MH1005
 U 1 1 5BD5294A
 P 3330 2260
-F 0 "MH?" H 3330 2460 50  0000 C CNN
+F 0 "MH1005" H 3330 2460 50  0000 C CNN
 F 1 "MountingHole" H 3330 2385 50  0000 C CNN
 F 2 "" H 3330 2260 50  0001 C CNN
@@
 $EndComp
 $Comp
-L Mechanical:MountingHole MH?
+L Mechanical:MountingHole MH1002
 U 1 1 5BD52A0A
 P 1830 3010
-F 0 "MH?" H 1830 3210 50  0000 C CNN
+F 0 "MH1002" H 1830 3210 50  0000 C CNN
 F 1 "MountingHole" H 1830 3135 50  0000 C CNN
 F 2 "" H 1830 3010 50  0001 C CNN
@@
 $EndComp
 $Comp
-L Mechanical:MountingHole MH?
+L Mechanical:MountingHole MH1004
 U 1 1 5BD52A11
 P 2580 3010
-F 0 "MH?" H 2580 3210 50  0000 C CNN
+F 0 "MH1004" H 2580 3210 50  0000 C CNN
 F 1 "MountingHole" H 2580 3135 50  0000 C CNN
 F 2 "" H 2580 3010 50  0001 C CNN
@@
 $EndComp
 $Comp
-L Mechanical:MountingHole MH?
+L Mechanical:MountingHole MH1006
 U 1 1 5BD52A18
 P 3330 3010
-F 0 "MH?" H 3330 3210 50  0000 C CNN
+F 0 "MH1006" H 3330 3210 50  0000 C CNN
 F 1 "MountingHole" H 3330 3135 50  0000 C CNN
 F 2 "" H 3330 3010 50  0001 C CNN

Commit message: Assigned footprints
Parts:
- MH1001, MH1002, MH1003, MH1004, MH1005, MH1006: footprint (none) -> Mounting_Holes:MountingHole_3mm
Changed lines of the file:
@@
 F 0 "MH1001" H 1830 2460 50  0000 C CNN
 F 1 "MountingHole" H 1830 2385 50  0000 C CNN
-F 2 "" H 1830 2260 50  0001 C CNN
+F 2 "Mounting_Holes:MountingHole_3mm" H 1830 2260 50  0001 C CNN
 F 3 "~" H 1830 2260 50  0001 C CNN
 	1    1830 2260
@@
 F 0 "MH1003" H 2580 2460 50  0000 C CNN
 F 1 "MountingHole" H 2580 2385 50  0000 C CNN
-F 2 "" H 2580 2260 50  0001 C CNN
+F 2 "Mounting_Holes:MountingHole_3mm" H 2580 2260 50  0001 C CNN
 F 3 "~" H 2580 2260 50  0001 C CNN
 	1    2580 2260
@@
 F 0 "MH1005" H 3330 2460 50  0000 C CNN
 F 1 "MountingHole" H 3330 2385 50  0000 C CNN
-F 2 "" H 3330 2260 50  0001 C CNN
+F 2 "Mounting_Holes:MountingHole_3mm" H 3330 2260 50  0001 C CNN
 F 3 "~" H 3330 2260 50  0001 C CNN
 	1    3330 2260
@@
 F 0 "MH1002" H 1830 3210 50  0000 C CNN
 F 1 "MountingHole" H 1830 3135 50  0000 C CNN
-F 2 "" H 1830 3010 50  0001 C CNN
+F 2 "Mounting_Holes:MountingHole_3mm" H 1830 3010 50  0001 C CNN
 F 3 "~" H 1830 3010 50  0001 C CNN
 	1    1830 3010
@@
 F 0 "MH1004" H 2580 3210 50  0000 C CNN
 F 1 "MountingHole" H 2580 3135 50  0000 C CNN
-F 2 "" H 2580 3010 50  0001 C CNN
+F 2 "Mounting_Holes:MountingHole_3mm" H 2580 3010 50  0001 C CNN
 F 3 "~" H 2580 3010 50  0001 C CNN
 	1    2580 3010
@@
 F 0 "MH1006" H 3330 3210 50  0000 C CNN
 F 1 "MountingHole" H 3330 3135 50  0000 C CNN
-F 2 "" H 3330 3010 50  0001 C CNN
+F 2 "Mounting_Holes:MountingHole_3mm" H 3330 3010 50  0001 C CNN
 F 3 "~" H 3330 3010 50  0001 C CNN
 	1    3330 3010

Commit message: A lot more power flooding
Parts:
- removed MH1003, MH1004: MountingHole, Mounting_Holes:MountingHole_3mm, symbol Mechanical:MountingHole
- removed MK1005, MK1006: 4-40 Screw, symbol Custom_Library:Screw
- removed MK1007, MK1008: 4-40 Standoff, symbol Custom_Library:Standoff
Changed lines of the file:
@@
-$EndComp
-$Comp
-L Custom_Library:Screw MK1005
-U 1 1 5BC1118A
-P 7220 2210
-F 0 "MK1005" H 7220 2310 50  0000 C CNN
-F 1 "4-40 Screw" H 7220 2410 50  0000 C CNN
-F 2 "" H 7220 2460 50  0001 C CNN
-F 3 "" H 7220 2460 50  0001 C CNN
-F 4 "36-9900-ND" H 0   0   50  0001 C CNN "Digi-Key PN"
-	1    7220 2210
-	1    0    0    -1
 $EndComp
 $Comp
@@
 F 4 "36-9900-ND" H 0   0   50  0001 C CNN "Digi-Key PN"
 	1    6470 2960
-	1    0    0    -1
-$EndComp
-$Comp
-L Custom_Library:Screw MK1006
-U 1 1 5BC113F5
-P 7220 2960
-F 0 "MK1006" H 7220 3060 50  0000 C CNN
-F 1 "4-40 Screw" H 7220 3160 50  0000 C CNN
-F 2 "" H 7220 3210 50  0001 C CNN
-F 3 "" H 7220 3210 50  0001 C CNN
-F 4 "36-9900-ND" H 0   0   50  0001 C CNN "Digi-Key PN"
-	1    7220 2960
 	1    0    0    -1
 $EndComp
@@
 $EndComp
 $Comp
-L Custom_Library:Standoff MK1007
-U 1 1 5BC12310
-P 7220 3720
-F 0 "MK1007" H 7220 3870 50  0000 C CNN
-F 1 "4-40 Standoff" H 7220 3970 50  0000 C CNN
-F 2 "" H 7220 4070 50  0001 C CNN
-F 3 "" H 7220 4070 50  0001 C CNN
-F 4 "36-8400-ND" H 0   0   50  0001 C CNN "Digi-Key PN"
-	1    7220 3720
-	1    0    0    -1
-$EndComp
-$Comp
 L Custom_Library:Standoff MK1011
 U 1 1 5BC1235A
@@
 F 4 "36-8400-ND" H 0   0   50  0001 C CNN "Digi-Key PN"
 	1    6470 4470
-	1    0    0    -1
-$EndComp
-$Comp
-L Custom_Library:Standoff MK1008
-U 1 1 5BC1253B
-P 7220 4470
-F 0 "MK1008" H 7220 4620 50  0000 C CNN
-F 1 "4-40 Standoff" H 7220 4720 50  0000 C CNN
-F 2 "" H 7220 4820 50  0001 C CNN
-F 3 "" H 7220 4820 50  0001 C CNN
-F 4 "36-8400-ND" H 0   0   50  0001 C CNN "Digi-Key PN"
-	1    7220 4470
 	1    0    0    -1
 $EndComp
@@
 $EndComp
 $Comp
-L Mechanical:MountingHole MH1003
-U 1 1 5BD52910
-P 2580 2260
-F 0 "MH1003" H 2580 2460 50  0000 C CNN
-F 1 "MountingHole" H 2580 2385 50  0000 C CNN
-F 2 "Mounting_Holes:MountingHole_3mm" H 2580 2260 50  0001 C CNN
-F 3 "~" H 2580 2260 50  0001 C CNN
-	1    2580 2260
-	1    0    0    -1
-$EndComp
-$Comp
 L Mechanical:MountingHole MH1005
 U 1 1 5BD5294A
@@
 	1    0    0    -1
 $EndComp
-$Comp
-L Mechanical:MountingHole MH1004
-U 1 1 5BD52A11
-P 2580 3010
-F 0 "MH1004" H 2580 3210 50  0000 C CNN
-F 1 "MountingHole" H 2580 3135 50  0000 C CNN
-F 2 "Mounting_Holes:MountingHole_3mm" H 2580 3010 50  0001 C CNN
-F 3 "~" H 2580 3010 50  0001 C CNN
-	1    2580 3010
-	1    0    0    -1
-$EndComp

Commit message: Resolved mounting hole ref des issue
Parts:
- renumbered MH1005 to MH1003, MH1002 to MH1004
Changed lines of the file:
@@
 $EndComp
 $Comp
-L Mechanical:MountingHole MH1005
+L Mechanical:MountingHole MH1003
 U 1 1 5BD5294A
 P 3330 2260
-F 0 "MH1005" H 3330 2460 50  0000 C CNN
+F 0 "MH1003" H 3330 2460 50  0000 C CNN
 F 1 "MountingHole" H 3330 2385 50  0000 C CNN
 F 2 "Mounting_Holes:MountingHole_3mm" H 3330 2260 50  0001 C CNN
@@
 $EndComp
 $Comp
-L Mechanical:MountingHole MH1002
+L Mechanical:MountingHole MH1004
 U 1 1 5BD52A0A
 P 1830 3010
-F 0 "MH1002" H 1830 3210 50  0000 C CNN
+F 0 "MH1004" H 1830 3210 50  0000 C CNN
 F 1 "MountingHole" H 1830 3135 50  0000 C CNN
 F 2 "Mounting_Holes:MountingHole_3mm" H 1830 3010 50  0001 C CNN
