File: hdw/LTC7851_Demo/Active_Load_1.sch (KiCad schematic (older format))
At the start: 16 parts, among them J1101 FG_LOAD, J1102 ISNS, Q1101 BSC123N10LSGATMA1, Q1102 BSC123N10LSGATMA1, U1101 LT1010DD

Commit message: Added a few connectors and cleaned up some routing
Parts:
- Q1101, Q1102: value BSC123N10LSGATMA1 -> IPC100N04S51R7ATMA1
Changed lines of the file:
@@
 P 7900 2420
 F 0 "Q1101" H 8100 2495 50  0000 L CNN
-F 1 "BSC123N10LSGATMA1" H 8100 2420 50  0000 L CNN
+F 1 "IPC100N04S51R7ATMA1" H 8100 2420 50  0000 L CNN
 F 2 "TO_SOT_Packages_SMD:TDSON-8-1" H 8100 2345 50  0001 L CIN
 F 3 "http://www.infineon.com/dgdl/Infineon-BSC123N10LS-DS-v02_08-en.pdf?fileId=db3a30431b3e89eb011b4626974b7df5" V 7900 2420 50  0001 L CNN
@@
 P 7900 4460
 F 0 "Q1102" H 8100 4535 50  0000 L CNN
-F 1 "BSC123N10LSGATMA1" H 8100 4460 50  0000 L CNN
+F 1 "IPC100N04S51R7ATMA1" H 8100 4460 50  0000 L CNN
 F 2 "TO_SOT_Packages_SMD:TDSON-8-1" H 8100 4385 50  0001 L CIN
 F 3 "http://www.infineon.com/dgdl/Infineon-BSC123N10LS-DS-v02_08-en.pdf?fileId=db3a30431b3e89eb011b4626974b7df5" V 7900 4460 50  0001 L CNN
