File: hdw/LTC7851_Demo/Active_Load_2.sch (KiCad schematic (older format))
At the start: 8 parts, among them Q1201 BSC123N10LSGATMA1, Q1202 BSC123N10LSGATMA1

Commit message: Added a few connectors and cleaned up some routing
Parts:
- Q1201, Q1202: value BSC123N10LSGATMA1 -> IPC100N04S51R7ATMA1
Changed lines of the file:
@@
 P 7900 2420
 F 0 "Q1201" H 8100 2495 50  0000 L CNN
-F 1 "BSC123N10LSGATMA1" H 8100 2420 50  0000 L CNN
+F 1 "IPC100N04S51R7ATMA1" H 8100 2420 50  0000 L CNN
 F 2 "TO_SOT_Packages_SMD:TDSON-8-1" H 8100 2345 50  0001 L CIN
 F 3 "http://www.infineon.com/dgdl/Infineon-BSC123N10LS-DS-v02_08-en.pdf?fileId=db3a30431b3e89eb011b4626974b7df5" V 7900 2420 50  0001 L CNN
@@
 P 7900 4460
 F 0 "Q1202" H 8100 4535 50  0000 L CNN
-F 1 "BSC123N10LSGATMA1" H 8100 4460 50  0000 L CNN
+F 1 "IPC100N04S51R7ATMA1" H 8100 4460 50  0000 L CNN
 F 2 "TO_SOT_Packages_SMD:TDSON-8-1" H 8100 4385 50  0001 L CIN
 F 3 "http://www.infineon.com/dgdl/Infineon-BSC123N10LS-DS-v02_08-en.pdf?fileId=db3a30431b3e89eb011b4626974b7df5" V 7900 4460 50  0001 L CNN
