File: hdw/LTC7851_Demo/LTC7851_Demo.kicad_pcb (KiCad board)
At the start: 4 copper layers, 100 x 50 mm, 199 parts, among them J1101 FG_LOAD, J1102 ISNS, J1401 VOUT, J1402 LOOP_TAP, J1403 Wave_Gen_In, J201 +12V IN, J206 GND IN, J301 CLKOUT, J302 RUN, J303 THDN, J304 IAVG, J305 PGOOD, J901 +5V OUT, J902 +5V OUT, J903 GND OUT, J904 GND OUT, Q1101 IPC100N04S51R7ATMA1, Q1102 IPC100N04S51R7ATMA1, Q1201 IPC100N04S51R7ATMA1, Q1202 IPC100N04S51R7ATMA1, Q1301 IPC100N04S51R7ATMA1, Q1302 IPC100N04S51R7ATMA1, Q201 IPC100N04S51R7ATMA1, Q202 IPC100N04S51R7ATMA1, T1401 1:1 Pulse Transformer, U1101 LT1010DD, U201 LTC4365DDB, U202 74LVC1G06, U301 LTC7851UHH, U302 74LVC1G17, U303 74LVC1G06, U304 74LVC1G06, U401 SiC779, U501 SiC779, U601 SiC779, U701 SiC779, U801 LM1117-ADJ

Commit message: Substantial wiring and layout changes
Parts:
- added R412: 0, Resistors_SMD:R_0402, F.Cu at (119.0, 98.1)
- added R413: 0, Resistors_SMD:R_0402, F.Cu at (119.0, 99.3)
- added R414: 0, Resistors_SMD:R_0402, F.Cu at (97.2, 98.5)
- added R504: 0, Resistors_SMD:R_0402, F.Cu at (136.3, 98.1)
- added R505: 0, Resistors_SMD:R_0402, F.Cu at (136.3, 99.3)
- added R604: 0, Resistors_SMD:R_0402, F.Cu at (153.8, 98.1)
- added R605: 0, Resistors_SMD:R_0402, F.Cu at (153.8, 99.3)
- added R704: 0, Resistors_SMD:R_0402, F.Cu at (171.1, 98.1)
- added R705: 0, Resistors_SMD:R_0402, F.Cu at (171.1, 99.3)
- C401, C403, C404, C406: footprint Capacitors_SMD:C_0603 -> Capacitors_SMD:C_0402
- C402: footprint Capacitors_SMD:C_0603 -> Capacitors_SMD:C_0402; moved to F.Cu
- C415, C510, C610, C710: footprint Capacitors_SMD:C_0603 -> Capacitors_SMD:C_0402; moved to B.Cu
- R401, R403, R404, R408, R409: footprint Resistors_SMD:R_0603 -> Resistors_SMD:R_0402
- R402: value 320 -> 324; footprint Resistors_SMD:R_0603 -> Resistors_SMD:R_0402
- R407, R410, R411, R503, R603, R703: footprint Resistors_SMD:R_0603 -> Resistors_SMD:R_0402; moved to B.Cu
- moved R410 47.7 mm to (140.9, 77.0)
- moved R411 47.7 mm to (142.1, 77.0), turned to 270 degrees
- moved C710 37.0 mm to (148.5, 70.3)
- moved R703 34.0 mm to (149.7, 70.3), turned to 90 degrees
- moved C415 34.0 mm to (141.7, 70.3)
- moved R407 33.8 mm to (140.5, 70.3), turned to 90 degrees
- moved C610 26.5 mm to (148.5, 72.2), turned to 180 degrees
- moved C510 25.6 mm to (141.5, 72.2), turned to 0 degrees
- moved R603 23.9 mm to (148.5, 73.3), turned to 180 degrees
- moved R503 23.8 mm to (141.5, 73.3)
- moved R408 4.47 mm to (99.8, 98.5)
- moved R402 3.90 mm to (141.2, 80.6)
- moved C403 3.78 mm to (142.4, 80.8)
- moved R404 3.06 mm to (141.9, 79.2)
- moved C401 2.73 mm to (151.1, 74.6), turned to 90 degrees
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Connections:
- net /POS5 Phase 1/POS5_VSNS1_+ renamed Net-(R410-Pad2)
- C401 pad 1: POS5_SS -> GND
- C401 pad 2: GND -> POS5_SS
- C402 pad 1: POS5_IAVG -> GND
- C402 pad 2: GND -> POS5_IAVG
- C415 pad 1: +5V -> /POS5 Phase 1/POS5_ISNS1_-
- C415 pad 2: /POS5 Phase 1/POS5_ISNS1_+ -> Net-(C415-Pad2)
- C510 pad 1: +5V -> /POS5 Phase 2/POS5_ISNS2_-
- C510 pad 2: /POS5 Phase 2/POS5_ISNS2_+ -> Net-(C510-Pad2)
- C610 pad 1: +5V -> /POS5 Phase 3/POS5_ISNS3_-
- C610 pad 2: /POS5 Phase 3/POS5_ISNS3_+ -> Net-(C610-Pad2)
- C710 pad 1: +5V -> /POS5 Phase 4/POS5_ISNS4_-
- C710 pad 2: /POS5 Phase 4/POS5_ISNS4_+ -> Net-(C710-Pad2)
- R407 pad 1: Net-(L401-Pad1) -> /POS5 Phase 1/POS5_ISNS1_+
- R407 pad 2: /POS5 Phase 1/POS5_ISNS1_+ -> Net-(C415-Pad2)
- R408 pad 1: GND -> /POS5 Phase 1/POS5_VSNSO1_-
- R408 pad 2: /POS5 Phase 1/POS5_VSNS1_- -> GND
- R409 pad 2: LOOP_TAP -> /POS5 Phase 1/POS5_VSNSO1_+
- R410 pad 1: LOOP_TAP -> /POS5 Phase 1/POS5_VSNSO1_+
- R411 pad 2: GND -> /POS5 Phase 1/POS5_VSNSO1_-
- R503 pad 1: Net-(L501-Pad1) -> /POS5 Phase 2/POS5_ISNS2_+
- R503 pad 2: /POS5 Phase 2/POS5_ISNS2_+ -> Net-(C510-Pad2)
- R603 pad 1: Net-(L601-Pad1) -> /POS5 Phase 3/POS5_ISNS3_+
- R603 pad 2: /POS5 Phase 3/POS5_ISNS3_+ -> Net-(C610-Pad2)
- R703 pad 1: Net-(L701-Pad1) -> /POS5 Phase 4/POS5_ISNS4_+
- R703 pad 2: /POS5 Phase 4/POS5_ISNS4_+ -> Net-(C710-Pad2)
- U301 pad 3: /POS5 Phase 1/POS5_VSNS1_- -> /POS5 Phase 1/POS5_VSNSO1_-
- U301 pad 31: /POS5 Phase 4/POS5_ISNS4_+ -> Net-(C710-Pad2)
- U301 pad 32: +5V -> /POS5 Phase 4/POS5_ISNS4_-
- U301 pad 33: +5V -> /POS5 Phase 3/POS5_ISNS3_-
- U301 pad 34: /POS5 Phase 3/POS5_ISNS3_+ -> Net-(C610-Pad2)
- U301 pad 43: /POS5 Phase 2/POS5_ISNS2_+ -> Net-(C510-Pad2)
- U301 pad 44: +5V -> /POS5 Phase 2/POS5_ISNS2_-
- U301 pad 45: +5V -> /POS5 Phase 1/POS5_ISNS1_-
- U301 pad 46: /POS5 Phase 1/POS5_ISNS1_+ -> Net-(C415-Pad2)
Routing:
- net +5V: track 265.7 -> 74.7 mm, vias 152 -> 143
- net /POS5 Phase 1/POS5_VSNSO1_-: track 0.00 -> 69.7 mm, vias 0 -> 5
- net /POS5 Phase 1/POS5_VSNS1_-: track 69.5 -> 0.00 mm, vias 4 -> 0
- net /POS5 Phase 1/POS5_VSNSO1_+: track 0.00 -> 67.7 mm, vias 0 -> 4
- net Net-(R410-Pad2): track 71.9 -> 4.30 mm, vias 2 -> 1
- net /POS5 Phase 4/POS5_ISNS4_-: track 0.00 -> 61.4 mm, vias 0 -> 3
- net /POS5 Phase 1/POS5_ISNS1_-: track 0.00 -> 46.6 mm, vias 0 -> 4
- net /POS5 Phase 2/POS5_ISNS2_-: track 0.00 -> 42.0 mm, vias 0 -> 2
- net /POS5 Phase 3/POS5_ISNS3_-: track 0.00 -> 40.6 mm, vias 0 -> 3
- net POS5_RUN: track 59.5 -> 47.0 mm
- net POS5_SS: track 37.1 -> 25.4 mm, vias 4 -> 3
- net /POS5 Phase 2/POS5_ISNS2_+: track 43.9 -> 34.4 mm, vias 2 -> 1
- net /POS5 Phase 4/POS5_ISNS4_+: track 49.8 -> 57.8 mm
- net POS5_PGOOD_OC: track 60.5 -> 67.8 mm, vias 9 -> 7
- net Net-(C610-Pad2): track 0.00 -> 6.09 mm, vias 0 -> 1
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
Commit message: Furthe rrouting refinements
Parts:
- added G***: Heat_Caution_Symbol, Custom Footprints Library:Heat_Caution_Symbol, F.Cu at (86.3, 72.3)
- added G***: Heat_Caution_Symbol, Custom Footprints Library:Heat_Caution_Symbol, F.Cu at (143.9, 84.2)
- added G***: Heat_Caution_Symbol, Custom Footprints Library:Heat_Caution_Symbol, B.Cu at (96.3, 103.4)
- added G***: MU_Logo_Silk, Custom Footprints Library:MU_Logo_Silk, B.Cu at (98.6, 85.4)
- added G***: Heat_Caution_Symbol, Custom Footprints Library:Heat_Caution_Symbol, B.Cu at (160.2, 91.6)
- added REF***: ESD-Logo_6.6x6mm_SilkScreen, Symbols:ESD-Logo_6.6x6mm_SilkScreen, F.Cu at (162.3, 84.3)
- added REF***: ESD-Logo_6.6x6mm_SilkScreen, Symbols:ESD-Logo_6.6x6mm_SilkScreen, B.Cu at (153.5, 72.2)
- added REF***: OSHW-Logo_5.7x6mm_SilkScreen, Symbols:OSHW-Logo_5.7x6mm_SilkScreen, B.Cu at (112.8, 89.4)
- moved C801 0.25 mm to (107.2, 91.0)
- moved C805 0.25 mm to (103.6, 91.0)
Routing:
- net Net-(U301-Pad24): track 40.9 -> 39.1 mm
- net /POS5 Phase 1/POS5_ISNS1_-: track 46.6 -> 47.9 mm
- net /POS5 Phase 1/POS5_ISNS1_+: track 41.9 -> 43.2 mm
- net +5.5V_MNG: track 55.2 -> 56.2 mm
- net GND: track 112.3 -> 113.2 mm
- net POS5_PGOOD_OC: track 67.8 -> 68.4 mm
- net +12V: track 72.2 -> 72.0 mm, vias 441 -> 442
Other:
- board text added: "LED Display Power Supply 1MHz 5V 80A Quad Phase Buck LTC7851 Voltage Mode Controller"
- board text removed: "LTC7851 Demo Board Four Phase 1MHz 5V 80A Buck"

Commit message: Finished routing and added 3D renders
Routing:
- net GND: track 113.2 -> 113.8 mm, vias 675 -> 683
